Commit message: いろいろやった

File: urdf/demorobot.urdf.xacro (robot description, xacro)
@@ -13,29 +13,18 @@
       <pose>0.1 0 0 0 0 0</pose>
       <mass value="${base_mass}"/>
-      <inertia>
-        <ixx>4.2111447e-02</ixx>
-        <ixy>0</ixy>
-        <ixz>0</ixz>
-        <iyy>4.2111447e-02</iyy>
-        <iyz>0</iyz>
-        <izz>7.5254874e-02</izz>
-      </inertia>
+      <inertia ixx="4.2111447e-02" ixy="0" ixz="0" iyy="4.2111447e-02" iyz="0" izz="7.5254874e-02"/>
     </inertial>
     <collision name="base_collision">
-      <pose>-0.064 0.08 0.06 0 0 -1.57</pose>
+      <pose>0 0 0 0 0 0</pose>
       <geometry>
-        <mesh>
-          <uri>model://meshes/2DRoboPrac.stl</uri>
-        </mesh>
+        <mesh filename="model://meshes/2DRoboPrac.stl"/>
       </geometry>
     </collision>
     <visual name="base_visual">
-      <pose>-0.064 0.08 0.06 0 0 -1.57</pose>
+      <pose>0 0 0 0 0 0</pose>
       <geometry>
-        <mesh>
-          <uri>model://meshes/2DRoboPrac.dae</uri>
-        </mesh>
+        <mesh filename="model://meshes/2DRoboPrac.dae"/>
       </geometry>
-      <material>
+      <material name="base_material">
         <color rgba="0.921568627 0.925490196 0.941176471 1"/>
       </material>
@@ -46,29 +35,16 @@
     <inertial>
       <mass value="${wheel_mass}"/>
-      <inertia>
-        <ixx>1.1175580e-05</ixx>
-        <ixy>-4.2369783e-11</ixy>
-        <ixz>-5.9381719e-09</ixz>
-        <iyy>1.1192413e-05</iyy>
-        <iyz>-1.4400107e-11</iyz>
-        <izz>2.0712558e-05</izz>
-      </inertia>
+      <inertia ixx="1.1175580e-05" ixy="-4.2369783e-11" ixz="-5.9381719e-09" iyy="1.1192413e-05" iyz="-1.4400107e-11" izz="2.0712558e-05"/>
     </inertial>
     <collision name="wheel_left_collision">
       <geometry>
-        <cylinder>
-          <radius>${wheel_radius}</radius>
-          <length>${wheel_length}</length>
-        </cylinder>
+        <cylinder radius="${wheel_radius}" length="${wheel_length}"/>
       </geometry>
     </collision>
     <visual name="wheel_left_visual">
       <geometry>
-        <cylinder>
-          <radius>${wheel_radius}</radius>
-          <length>${wheel_length}</length>
-        </cylinder>
+        <cylinder radius="${wheel_radius}" length="${wheel_length}"/>
       </geometry>
-      <material>
+      <material name="wheel_material">
         <color rgba="1.0 0.0 0.0 1"/>
       </material>
@@ -87,29 +63,16 @@
     <inertial>
       <mass value="${wheel_mass}"/>
-      <inertia>
-        <ixx>1.1175580e-05</ixx>
-        <ixy>-4.2369783e-11</ixy>
-        <ixz>-5.9381719e-09</ixz>
-        <iyy>1.1192413e-05</iyy>
-        <iyz>-1.4400107e-11</iyz>
-        <izz>2.0712558e-05</izz>
-      </inertia>
+      <inertia ixx="1.1175580e-05" ixy="-4.2369783e-11" ixz="-5.9381719e-09" iyy="1.1192413e-05" iyz="-1.4400107e-11" izz="2.0712558e-05"/>
     </inertial>
     <collision name="wheel_right_collision">
       <geometry>
-        <cylinder>
-          <radius>${wheel_radius}</radius>
-          <length>${wheel_length}</length>
-        </cylinder>
+        <cylinder radius="${wheel_radius}" length="${wheel_length}"/>
       </geometry>
     </collision>
     <visual name="wheel_right_visual">
       <geometry>
-        <cylinder>
-          <radius>${wheel_radius}</radius>
-          <length>${wheel_length}</length>
-        </cylinder>
+        <cylinder radius="${wheel_radius}" length="${wheel_length}"/>
       </geometry>
-      <material>
+      <material name="wheel_material">
         <color rgba="1.0 0.0 0.0 1"/>
       </material>
@@ -128,35 +91,26 @@
     <inertial>
       <mass value="${caster_mass}"/>
-      <inertia>
-        <ixx>0.00001</ixx>
-        <ixy>0.000</ixy>
-        <ixz>0.000</ixz>
-        <iyy>0.00001</iyy>
-        <iyz>0.000</iyz>
-        <izz>0.00001</izz>
-      </inertia>
+      <inertia ixx="0.00001" ixy="0.000" ixz="0.000" iyy="0.00001" iyz="0.000" izz="0.00001"/>
     </inertial>
     <collision name="caster_back_right_collision">
       <geometry>
-        <sphere>
-          <radius>0.005</radius>
-        </sphere>
+        <sphere radius="0.005"/>
       </geometry>
     </collision>
     <visual name="caster_back_right_visual">
       <geometry>
-        <sphere>
-          <radius>0.005</radius>
-        </sphere>
+        <sphere radius="0.005"/>
       </geometry>
-      <material>
+      <material name="caster_material">
         <color rgba="0.0 1.0 0.0 1"/>
       </material>
     </visual>
   </link>
-  <joint name="caster_back_right_joint" type="ball">
+  <joint name="caster_back_right_joint" type="fixed">
     <parent link="base_link"/>
     <child link="caster_back_right_link"/>
     <origin xyz="0.15 -0.05 -0.004" rpy="-1.57 0 0"/>
+    <axis xyz="0 0 1"/>
+    <limit effort="1" velocity="10" lower="-3.14159" upper="3.14159"/>
   </joint>
   <!-- Caster wheels (back left) -->
@@ -164,40 +118,31 @@
     <inertial>
       <mass value="${caster_mass}"/>
-      <inertia>
-        <ixx>0.00001</ixx>
-        <ixy>0.000</ixy>
-        <ixz>0.000</ixz>
-        <iyy>0.00001</iyy>
-        <iyz>0.000</iyz>
-        <izz>0.00001</izz>
-      </inertia>
+      <inertia ixx="0.00001" ixy="0.000" ixz="0.000" iyy="0.00001" iyz="0.000" izz="0.00001"/>
     </inertial>
     <collision name="caster_back_left_collision">
       <geometry>
-        <sphere>
-          <radius>0.005</radius>
-        </sphere>
+        <sphere radius="0.005"/>
       </geometry>
     </collision>
     <visual name="caster_back_left_visual">
       <geometry>
-        <sphere>
-          <radius>0.005</radius>
-        </sphere>
+        <sphere radius="0.005"/>
       </geometry>
-      <material>
+      <material name="caster_material">
         <color rgba="0.0 1.0 0.0 1"/>
       </material>
     </visual>
   </link>
-  <joint name="caster_back_left_joint" type="ball">
+  <joint name="caster_back_left_joint" type="fixed">
     <parent link="base_link"/>
     <child link="caster_back_left_link"/>
     <origin xyz="0.15 0.05 -0.004" rpy="-1.57 0 0"/>
+    <axis xyz="0 0 1"/>
+    <limit effort="1" velocity="10" lower="-3.14159" upper="3.14159"/>
   </joint>
   <!-- ros2_control plugin config -->
   <ros2_control name="GazeboSystem" type="system">
     <hardware>
-      <plugin>gazebo_ros2_control/GazeboSystem</plugin>
+      <plugin>gz_ros2_control/GazeboSimSystem</plugin>
     </hardware>
     <joint name="wheel_left_joint">
@@ -219,6 +164,6 @@
   </ros2_control>
   <gazebo>
-    <plugin filename="libgazebo_ros2_control.so" name="gazebo_ros2_control">
-      <parameters>$(find gazebo_simulator)/config/ros2_controllers.yaml</parameters>
+    <plugin filename="libgz_ros2_control-system.so" name="gz_ros2_control::GazeboSimROS2ControlPlugin">
+      <parameters>$(find gazebo_simulator)/config/controller_config.yaml</parameters>
     </plugin>
   </gazebo>

Commit message: 差動2輪。それぞれのモーターで動いた。

File: urdf/demorobot.urdf.xacro (robot description, xacro)
@@ -16,5 +16,5 @@
     </inertial>
     <collision name="base_collision">
-      <pose>0 0 0 0 0 0</pose>
+      <origin xyz="-0.064 0.08 0.06" rpy="0 0 -1.57"/>
       <geometry>
         <mesh filename="model://meshes/2DRoboPrac.stl"/>
@@ -22,5 +22,5 @@
     </collision>
     <visual name="base_visual">
-      <pose>0 0 0 0 0 0</pose>
+      <origin xyz="-0.064 0.08 0.06" rpy="0 0 -1.57"/>
       <geometry>
         <mesh filename="model://meshes/2DRoboPrac.dae"/>
@@ -51,10 +51,10 @@
     </visual>
   </link>
-  <joint name="wheel_left_joint" type="revolute">
+  <joint name="wheel_left_joint" type="continuous">
     <parent link="base_link"/>
     <child link="wheel_left_link"/>
     <origin xyz="0.0 0.095 0.023" rpy="-1.57 0 0"/>
     <axis xyz="0 0 1"/>
-    <limit effort="10" velocity="10" lower="-3.14159" upper="3.14159"/>
+    <limit effort="10" velocity="10"/>
     <dynamics damping="0.0" friction="0.0"/>
   </joint>
@@ -79,10 +79,10 @@
     </visual>
   </link>
-  <joint name="wheel_right_joint" type="revolute">
+  <joint name="wheel_right_joint" type="continuous">
     <parent link="base_link"/>
     <child link="wheel_right_link"/>
     <origin xyz="0.0 -0.095 0.023" rpy="-1.57 0 0"/>
     <axis xyz="0 0 1"/>
-    <limit effort="10" velocity="10" lower="-3.14159" upper="3.14159"/>
+    <limit effort="10" velocity="10"/>
     <dynamics damping="0.0" friction="0.0"/>
   </joint>
@@ -112,5 +112,5 @@
     <origin xyz="0.15 -0.05 -0.004" rpy="-1.57 0 0"/>
     <axis xyz="0 0 1"/>
-    <limit effort="1" velocity="10" lower="-3.14159" upper="3.14159"/>
+    <limit effort="10" velocity="100" lower="-30.14159" upper="30.14159"/>
   </joint>
   <!-- Caster wheels (back left) -->
@@ -139,5 +139,5 @@
     <origin xyz="0.15 0.05 -0.004" rpy="-1.57 0 0"/>
     <axis xyz="0 0 1"/>
-    <limit effort="1" velocity="10" lower="-3.14159" upper="3.14159"/>
+    <limit effort="10" velocity="100" lower="-30.14159" upper="30.14159"/>
   </joint>
   <!-- ros2_control plugin config -->
@@ -148,6 +148,7 @@
     <joint name="wheel_left_joint">
       <command_interface name="velocity">
-        <param name="min">-10</param>
-        <param name="max">10</param>
+      <!-- これ↓いみない制限やわ -->
+        <!-- <param name="min">-10</param>
+        <param name="max">10</param> -->
       </command_interface>
       <state_interface name="position"/>
@@ -156,6 +157,7 @@
     <joint name="wheel_right_joint">
       <command_interface name="velocity">
-        <param name="min">-10</param>
-        <param name="max">10</param>
+        <!-- これ↓いみない制限やわ -->
+        <!-- <param name="min">-10</param>
+        <param name="max">10</param> -->
       </command_interface>
       <state_interface name="position"/>

Commit message: おむにバレルありおためし

File: urdf/demorobot.urdf.xacro (robot description, xacro)
@@ -18,5 +18,5 @@
       <origin xyz="-0.064 0.08 0.06" rpy="0 0 -1.57"/>
       <geometry>
-        <mesh filename="model://meshes/2DRoboPrac.stl"/>
+        <mesh filename="model://demorobot/meshes/2DRoboPrac.stl"/>
       </geometry>
     </collision>
@@ -24,5 +24,5 @@
       <origin xyz="-0.064 0.08 0.06" rpy="0 0 -1.57"/>
       <geometry>
-        <mesh filename="model://meshes/2DRoboPrac.dae"/>
+        <mesh filename="model://demorobot/meshes/2DRoboPrac.dae"/>
       </geometry>
       <material name="base_material">

File: urdf/omni4.urdf.xacro (robot description, xacro)
@@ -1,5 +1,5 @@
 <?xml version="1.0"?>
 <robot xmlns:xacro="http://www.ros.org/wiki/xacro" name="omni4_robot">
-  <!-- Parameters -->
+  <!-- Use visual meshes from sim2_lecture's omni wheel set while keeping simple controllable joints -->
   <xacro:property name="wheel_radius" value="0.033"/>
   <xacro:property name="wheel_width" value="0.018"/>
@@ -28,6 +28,7 @@
     </collision>
   </link>
-  <!-- Wheel link macro -->
-  <xacro:macro name="omni_wheel" params="name x y">
+  <!-- Per-wheel: a simple controllable revolute joint + visual from odm meshes -->
+  <xacro:macro name="odm_visual_wheel" params="name x y mesh_housing mesh_barrel">
+    <!-- controlled rotor link -->
     <link name="${name}_link">
       <inertial>
@@ -38,11 +39,10 @@
         <origin xyz="0 0 0" rpy="0 0 0"/>
         <geometry>
-          <cylinder radius="${wheel_radius}" length="${wheel_width}"/>
+          <!-- main housing mesh (optional) -->
+          <mesh filename="${mesh_housing}"/>
         </geometry>
-        <material name="wheel_material">
-          <color rgba="0.1 0.1 0.1 1"/>
-        </material>
       </visual>
       <collision>
+        <!-- keep simple cylinder collision for performance -->
         <geometry>
           <cylinder radius="${wheel_radius}" length="${wheel_width}"/>
@@ -59,10 +59,10 @@
     </joint>
   </xacro:macro>
-  <!-- Define four omni wheels (front_left, front_right, rear_left, rear_right) -->
-  <xacro:omni_wheel name="wheel_front_left" x="${wheel_x}" y="${wheel_y}"/>
-  <xacro:omni_wheel name="wheel_front_right" x="${wheel_x}" y="-${wheel_y}"/>
-  <xacro:omni_wheel name="wheel_rear_left" x="-${wheel_x}" y="${wheel_y}"/>
-  <xacro:omni_wheel name="wheel_rear_right" x="-${wheel_x}" y="-${wheel_y}"/>
-  <!-- ros2_control plugin config -->
+  <!-- Create four wheels using meshes from sim2_lecture if available -->
+  <xacro:odm_visual_wheel name="wheel_front_left" x="${wheel_x}" y="${wheel_y}" mesh_housing="package://sim2_lecture/stl/omni_housing.stl" mesh_barrel="package://sim2_lecture/stl/omni_barrel.stl"/>
+  <xacro:odm_visual_wheel name="wheel_front_right" x="${wheel_x}" y="-${wheel_y}" mesh_housing="package://sim2_lecture/stl/omni_housing.stl" mesh_barrel="package://sim2_lecture/stl/omni_barrel.stl"/>
+  <xacro:odm_visual_wheel name="wheel_rear_left" x="-${wheel_x}" y="${wheel_y}" mesh_housing="package://sim2_lecture/stl/omni_housing.stl" mesh_barrel="package://sim2_lecture/stl/omni_barrel.stl"/>
+  <xacro:odm_visual_wheel name="wheel_rear_right" x="-${wheel_x}" y="-${wheel_y}" mesh_housing="package://sim2_lecture/stl/omni_housing.stl" mesh_barrel="package://sim2_lecture/stl/omni_barrel.stl"/>
+  <!-- ros2_control plugin config (keep velocity interfaces compatible with existing controllers) -->
   <ros2_control name="GazeboSystem" type="system">
     <hardware>
@@ -70,7 +70,5 @@
     </hardware>
     <joint name="wheel_front_left_joint">
-    <!-- ここ↓をpositionにすると位置制御 -->
       <command_interface name="velocity"/>
-    <!-- ここ↓は返す値の種類 -->
       <state_interface name="position"/>
       <state_interface name="velocity"/>
