Commit message: 二輪車左の車輪を45°傾けた。うまく行った。

File: models/demorobot/demorobot.urdf (robot description, URDF)
Before this commit: robot demorobot, 5 links, 4 joints
Joints:
- joint wheel_left_joint: origin xyz=0.0 0.095 0.023 rpy=-1.57 0 0 -> xyz=0.0 0.095 0.023 rpy=-1.57 0 -0.7854

File: urdf/demorobot.urdf.xacro (robot description, xacro)
@@ -54,5 +54,5 @@
     <parent link="base_link"/>
     <child link="wheel_left_link"/>
-    <origin xyz="0.0 0.095 0.023" rpy="-1.57 0 0"/>
+    <origin xyz="0.0 0.095 0.023" rpy="-1.57 0 -0.7854"/>
     <axis xyz="0 0 1"/>
     <limit effort="10" velocity="10"/>

Commit message: もとの普通の2輪車に戻した

File: models/demorobot/demorobot.urdf (robot description, URDF)
Before this commit: robot demorobot, 5 links, 4 joints
Joints:
- joint wheel_left_joint: origin xyz=0.0 0.095 0.023 rpy=-1.57 0 -0.7854 -> xyz=0.0 0.095 0.023 rpy=-1.57 0 0

File: urdf/demorobot.urdf.xacro (robot description, xacro)
@@ -54,5 +54,5 @@
     <parent link="base_link"/>
     <child link="wheel_left_link"/>
-    <origin xyz="0.0 0.095 0.023" rpy="-1.57 0 -0.7854"/>
+    <origin xyz="0.0 0.095 0.023" rpy="-1.57 0 0"/>
     <axis xyz="0 0 1"/>
     <limit effort="10" velocity="10"/>
