Commit message: .yamlファイルを変更しやすいように改造

File: models/omni4/omni4.urdf (robot description, URDF)
Before this commit: robot omni4_robot, 5 links, 4 joints
Links:
- link wheel_front_left_link: geometry collision cylinder length=0.018 radius=0.033; visual mesh filename=package://sim2_lecture/stl/omni_housing.stl
- link wheel_front_right_link: geometry collision cylinder length=0.018 radius=0.033; visual mesh filename=package://sim2_lecture/stl/omni_housing.stl
- link wheel_rear_left_link: geometry collision cylinder length=0.018 radius=0.033; visual mesh filename=package://sim2_lecture/stl/omni_housing.stl
- link wheel_rear_right_link: geometry collision cylinder length=0.018 radius=0.033; visual mesh filename=package://sim2_lecture/stl/omni_housing.stl

Commit message: 一旦、omniはスポーンした。謎の物体すぎるけど

File: models/omni4/omni4.urdf (robot description, URDF)
Before this commit: robot omni4_robot, 5 links, 4 joints
Links:
- link wheel_front_left_link: geometry collision cylinder length=0.018 radius=0.033; visual mesh filename=model://omni4/meshes/omni_housing.stl
- link wheel_front_right_link: geometry collision cylinder length=0.018 radius=0.033; visual mesh filename=model://omni4/meshes/omni_housing.stl
- link wheel_rear_left_link: geometry collision cylinder length=0.018 radius=0.033; visual mesh filename=model://omni4/meshes/omni_housing.stl
- link wheel_rear_right_link: geometry collision cylinder length=0.018 radius=0.033; visual mesh filename=model://omni4/meshes/omni_housing.stl

File: urdf/omni4.urdf.xacro (robot description, xacro)
@@ -60,8 +60,8 @@
   </xacro:macro>
   <!-- Create four wheels using meshes from sim2_lecture if available -->
-  <xacro:odm_visual_wheel name="wheel_front_left" x="${wheel_x}" y="${wheel_y}" mesh_housing="package://sim2_lecture/stl/omni_housing.stl" mesh_barrel="package://sim2_lecture/stl/omni_barrel.stl"/>
-  <xacro:odm_visual_wheel name="wheel_front_right" x="${wheel_x}" y="-${wheel_y}" mesh_housing="package://sim2_lecture/stl/omni_housing.stl" mesh_barrel="package://sim2_lecture/stl/omni_barrel.stl"/>
-  <xacro:odm_visual_wheel name="wheel_rear_left" x="-${wheel_x}" y="${wheel_y}" mesh_housing="package://sim2_lecture/stl/omni_housing.stl" mesh_barrel="package://sim2_lecture/stl/omni_barrel.stl"/>
-  <xacro:odm_visual_wheel name="wheel_rear_right" x="-${wheel_x}" y="-${wheel_y}" mesh_housing="package://sim2_lecture/stl/omni_housing.stl" mesh_barrel="package://sim2_lecture/stl/omni_barrel.stl"/>
+  <xacro:odm_visual_wheel name="wheel_front_left" x="${wheel_x}" y="${wheel_y}" mesh_housing="model://omni4/meshes/omni_housing.stl" mesh_barrel="model://omni4/meshes/omni_barrel.stl"/>
+  <xacro:odm_visual_wheel name="wheel_front_right" x="${wheel_x}" y="-${wheel_y}" mesh_housing="model://omni4/meshes/omni_housing.stl" mesh_barrel="model://omni4/meshes/omni_barrel.stl"/>
+  <xacro:odm_visual_wheel name="wheel_rear_left" x="-${wheel_x}" y="${wheel_y}" mesh_housing="model://omni4/meshes/omni_housing.stl" mesh_barrel="model://omni4/meshes/omni_barrel.stl"/>
+  <xacro:odm_visual_wheel name="wheel_rear_right" x="-${wheel_x}" y="-${wheel_y}" mesh_housing="model://omni4/meshes/omni_housing.stl" mesh_barrel="model://omni4/meshes/omni_barrel.stl"/>
   <!-- ros2_control plugin config (keep velocity interfaces compatible with existing controllers) -->
   <ros2_control name="GazeboSystem" type="system">
@@ -92,5 +92,5 @@
   <gazebo>
     <plugin filename="libgz_ros2_control-system.so" name="gz_ros2_control::GazeboSimROS2ControlPlugin">
-      <parameters>$(find gazebo_simulator)/config/controller.yaml</parameters>
+      <parameters>$(find gazebo_simulator)/config/controller_omni4.yaml</parameters>
     </plugin>
   </gazebo>

Commit message: 4輪のむきがへん

File: models/omni4/omni4.urdf (robot description, URDF)
Before this commit: robot omni4_robot, 5 links, 4 joints
Joints:
- joint wheel_front_left_joint: origin xyz=0.12 0.095 0.02 rpy=0 0 1.5708 -> xyz=0.12 0.095 0.02 rpy=0 0 0
- joint wheel_front_right_joint: origin xyz=0.12 -0.095 0.02 rpy=0 0 1.5708 -> xyz=0.12 -0.095 0.02 rpy=0 0 0
- joint wheel_rear_left_joint: origin xyz=-0.12 0.095 0.02 rpy=0 0 1.5708 -> xyz=-0.12 0.095 0.02 rpy=0 0 0
- joint wheel_rear_right_joint: origin xyz=-0.12 -0.095 0.02 rpy=0 0 1.5708 -> xyz=-0.12 -0.095 0.02 rpy=0 0 0

File: urdf/omni4.urdf.xacro (robot description, xacro)
@@ -19,5 +19,7 @@
       </geometry>
       <material name="base_material">
-        <color rgba="0.8 0.8 0.8 1"/>
+        <!-- <color rgba="0.8 0.8 0.8 1"/> -->
+        <!-- ↓透明化↑普通 -->
+        <color rgba="1 1 1 0"/>
       </material>
     </visual>
@@ -37,5 +39,5 @@
       </inertial>
       <visual>
-        <origin xyz="0 0 0" rpy="0 0 0"/>
+        <origin xyz="0 0 0" rpy="0 1.5708 0"/>
         <geometry>
           <!-- main housing mesh (optional) -->
@@ -45,4 +47,5 @@
       <collision>
         <!-- keep simple cylinder collision for performance -->
+        <origin xyz="0 0 0" rpy="0 1.5708 0"/>
         <geometry>
           <cylinder radius="${wheel_radius}" length="${wheel_width}"/>
@@ -50,8 +53,12 @@
       </collision>
     </link>
+    <!-- 色 -->
+    <gazebo reference="${name}_link">
+      <material>Gazebo/Grey</material>
+    </gazebo>
     <joint name="${name}_joint" type="continuous">
       <parent link="base_link"/>
       <child link="${name}_link"/>
-      <origin xyz="${x} ${y} 0.02" rpy="0 0 1.5708"/>
+      <origin xyz="${x} ${y} 0.02" rpy="0 0 0"/>
       <axis xyz="0 0 1"/>
       <limit effort="10" velocity="20"/>

Commit message: 個別にrpyを設定はできた

File: models/omni4/omni4.urdf (robot description, URDF)
Before this commit: robot omni4_robot, 5 links, 4 joints
Joints:
- joint wheel_front_left_joint: origin xyz=0.12 0.095 0.02 rpy=0 0 0 -> xyz=0.12 0.095 0.02 rpy=0 0.785398 1.570796
- joint wheel_front_right_joint: origin xyz=0.12 -0.095 0.02 rpy=0 0 0 -> xyz=0.12 -0.095 0.02 rpy=0 0.785398 -0.785398
- joint wheel_rear_left_joint: origin xyz=-0.12 0.095 0.02 rpy=0 0 0 -> xyz=-0.12 0.095 0.02 rpy=0 -0.785398 -0.785398
- joint wheel_rear_right_joint: origin xyz=-0.12 -0.095 0.02 rpy=0 0 0 -> xyz=-0.12 -0.095 0.02 rpy=0 -0.785398 0.785398

File: urdf/omni4.urdf.xacro (robot description, xacro)
@@ -31,5 +31,5 @@
   </link>
   <!-- Per-wheel: a simple controllable revolute joint + visual from odm meshes -->
-  <xacro:macro name="odm_visual_wheel" params="name x y mesh_housing mesh_barrel">
+  <xacro:macro name="odm_visual_wheel" params="name x y r p yaw mesh_housing mesh_barrel">
     <!-- controlled rotor link -->
     <link name="${name}_link">
@@ -39,5 +39,5 @@
       </inertial>
       <visual>
-        <origin xyz="0 0 0" rpy="0 1.5708 0"/>
+        <origin xyz="0 0 0" rpy="${r} ${p} ${yaw}"/>
         <geometry>
           <!-- main housing mesh (optional) -->
@@ -47,5 +47,5 @@
       <collision>
         <!-- keep simple cylinder collision for performance -->
-        <origin xyz="0 0 0" rpy="0 1.5708 0"/>
+        <origin xyz="0 0 0" rpy="${r} ${p} ${yaw}"/>
         <geometry>
           <cylinder radius="${wheel_radius}" length="${wheel_width}"/>
@@ -60,5 +60,5 @@
       <parent link="base_link"/>
       <child link="${name}_link"/>
-      <origin xyz="${x} ${y} 0.02" rpy="0 0 0"/>
+      <origin xyz="${x} ${y} 0.02" rpy="${r} ${p} ${yaw}"/>
       <axis xyz="0 0 1"/>
       <limit effort="10" velocity="20"/>
@@ -67,8 +67,8 @@
   </xacro:macro>
   <!-- Create four wheels using meshes from sim2_lecture if available -->
-  <xacro:odm_visual_wheel name="wheel_front_left" x="${wheel_x}" y="${wheel_y}" mesh_housing="model://omni4/meshes/omni_housing.stl" mesh_barrel="model://omni4/meshes/omni_barrel.stl"/>
-  <xacro:odm_visual_wheel name="wheel_front_right" x="${wheel_x}" y="-${wheel_y}" mesh_housing="model://omni4/meshes/omni_housing.stl" mesh_barrel="model://omni4/meshes/omni_barrel.stl"/>
-  <xacro:odm_visual_wheel name="wheel_rear_left" x="-${wheel_x}" y="${wheel_y}" mesh_housing="model://omni4/meshes/omni_housing.stl" mesh_barrel="model://omni4/meshes/omni_barrel.stl"/>
-  <xacro:odm_visual_wheel name="wheel_rear_right" x="-${wheel_x}" y="-${wheel_y}" mesh_housing="model://omni4/meshes/omni_housing.stl" mesh_barrel="model://omni4/meshes/omni_barrel.stl"/>
+  <xacro:odm_visual_wheel name="wheel_front_left" x="${wheel_x}" y="${wheel_y}" r="0" p="0.785398" yaw="1.570796" mesh_housing="model://omni4/meshes/omni_housing.stl" mesh_barrel="model://omni4/meshes/omni_barrel.stl"/>
+  <xacro:odm_visual_wheel name="wheel_front_right" x="${wheel_x}" y="-${wheel_y}" r="0" p="0.785398" yaw="-0.785398" mesh_housing="model://omni4/meshes/omni_housing.stl" mesh_barrel="model://omni4/meshes/omni_barrel.stl"/>
+  <xacro:odm_visual_wheel name="wheel_rear_left" x="-${wheel_x}" y="${wheel_y}" r="0" p="-0.785398" yaw="-0.785398" mesh_housing="model://omni4/meshes/omni_housing.stl" mesh_barrel="model://omni4/meshes/omni_barrel.stl"/>
+  <xacro:odm_visual_wheel name="wheel_rear_right" x="-${wheel_x}" y="-${wheel_y}" r="0" p="-0.785398" yaw="0.785398" mesh_housing="model://omni4/meshes/omni_housing.stl" mesh_barrel="model://omni4/meshes/omni_barrel.stl"/>
   <!-- ros2_control plugin config (keep velocity interfaces compatible with existing controllers) -->
   <ros2_control name="GazeboSystem" type="system">

Commit message: まだ変。

File: models/omni4/omni4.urdf (robot description, URDF)
Before this commit: robot omni4_robot, 5 links, 4 joints
Joints:
- joint wheel_front_left_joint: origin xyz=0.12 0.095 0.02 rpy=0 0.785398 1.570796 -> xyz=0.12 0.095 0.02 rpy=1.570796 0 0.7854
- joint wheel_front_right_joint: origin xyz=0.12 -0.095 0.02 rpy=0 0.785398 -0.785398 -> xyz=0.12 -0.095 0.02 rpy=1.570796 0 -0.7854
- joint wheel_rear_left_joint: origin xyz=-0.12 0.095 0.02 rpy=0 -0.785398 -0.785398 -> xyz=-0.12 0.095 0.02 rpy=-1.570796 0 2.3562
- joint wheel_rear_right_joint: origin xyz=-0.12 -0.095 0.02 rpy=0 -0.785398 0.785398 -> xyz=-0.12 -0.095 0.02 rpy=-1.570796 0 -2.3562

File: urdf/omni4.urdf.xacro (robot description, xacro)
@@ -67,8 +67,8 @@
   </xacro:macro>
   <!-- Create four wheels using meshes from sim2_lecture if available -->
-  <xacro:odm_visual_wheel name="wheel_front_left" x="${wheel_x}" y="${wheel_y}" r="0" p="0.785398" yaw="1.570796" mesh_housing="model://omni4/meshes/omni_housing.stl" mesh_barrel="model://omni4/meshes/omni_barrel.stl"/>
-  <xacro:odm_visual_wheel name="wheel_front_right" x="${wheel_x}" y="-${wheel_y}" r="0" p="0.785398" yaw="-0.785398" mesh_housing="model://omni4/meshes/omni_housing.stl" mesh_barrel="model://omni4/meshes/omni_barrel.stl"/>
-  <xacro:odm_visual_wheel name="wheel_rear_left" x="-${wheel_x}" y="${wheel_y}" r="0" p="-0.785398" yaw="-0.785398" mesh_housing="model://omni4/meshes/omni_housing.stl" mesh_barrel="model://omni4/meshes/omni_barrel.stl"/>
-  <xacro:odm_visual_wheel name="wheel_rear_right" x="-${wheel_x}" y="-${wheel_y}" r="0" p="-0.785398" yaw="0.785398" mesh_housing="model://omni4/meshes/omni_housing.stl" mesh_barrel="model://omni4/meshes/omni_barrel.stl"/>
+  <xacro:odm_visual_wheel name="wheel_front_left" x="${wheel_x}" y="${wheel_y}" r="1.570796" p="0" yaw="0.7854" mesh_housing="model://omni4/meshes/omni_housing.stl" mesh_barrel="model://omni4/meshes/omni_barrel.stl"/>
+  <xacro:odm_visual_wheel name="wheel_front_right" x="${wheel_x}" y="-${wheel_y}" r="1.570796" p="0" yaw="-0.7854" mesh_housing="model://omni4/meshes/omni_housing.stl" mesh_barrel="model://omni4/meshes/omni_barrel.stl"/>
+  <xacro:odm_visual_wheel name="wheel_rear_left" x="-${wheel_x}" y="${wheel_y}" r="-1.570796" p="0" yaw="2.3562" mesh_housing="model://omni4/meshes/omni_housing.stl" mesh_barrel="model://omni4/meshes/omni_barrel.stl"/>
+  <xacro:odm_visual_wheel name="wheel_rear_right" x="-${wheel_x}" y="-${wheel_y}" r="-1.570796" p="0" yaw="-2.3562" mesh_housing="model://omni4/meshes/omni_housing.stl" mesh_barrel="model://omni4/meshes/omni_barrel.stl"/>
   <!-- ros2_control plugin config (keep velocity interfaces compatible with existing controllers) -->
   <ros2_control name="GazeboSystem" type="system">

Commit message: いろいろ実験

File: models/omni4/omni4.urdf (robot description, URDF)
Before this commit: robot omni4_robot, 5 links, 4 joints
Joints:
- joint wheel_front_left_joint: origin xyz=0.12 0.095 0.02 rpy=1.570796 0 0.7854 -> xyz=0.12 0.095 0.02 rpy=1.5708 0 -2.35619
- joint wheel_front_right_joint: origin xyz=0.12 -0.095 0.02 rpy=1.570796 0 -0.7854 -> xyz=0.12 -0.095 0.02 rpy=0 0 0
- joint wheel_rear_left_joint: origin xyz=-0.12 0.095 0.02 rpy=-1.570796 0 2.3562 -> xyz=-0.12 0.095 0.02 rpy=0 0 0
- joint wheel_rear_right_joint: origin xyz=-0.12 -0.095 0.02 rpy=-1.570796 0 -2.3562 -> xyz=-0.12 -0.095 0.02 rpy=0 0 0

File: urdf/omni4.urdf.xacro (robot description, xacro)
@@ -31,5 +31,5 @@
   </link>
   <!-- Per-wheel: a simple controllable revolute joint + visual from odm meshes -->
-  <xacro:macro name="odm_visual_wheel" params="name x y r p yaw mesh_housing mesh_barrel">
+  <xacro:macro name="odm_visual_wheel" params="name x y r p yaw mesh_housing mesh_barrel axis_x='0' axis_y='0' axis_z='1'">
     <!-- controlled rotor link -->
     <link name="${name}_link">
@@ -61,5 +61,5 @@
       <child link="${name}_link"/>
       <origin xyz="${x} ${y} 0.02" rpy="${r} ${p} ${yaw}"/>
-      <axis xyz="0 0 1"/>
+      <axis xyz="${axis_x} ${axis_y} ${axis_z}"/>
       <limit effort="10" velocity="20"/>
       <dynamics damping="0.0" friction="0.0"/>
@@ -67,8 +67,20 @@
   </xacro:macro>
   <!-- Create four wheels using meshes from sim2_lecture if available -->
+  <xacro:odm_visual_wheel name="wheel_front_left" x="${wheel_x}" y="${wheel_y}" r="0" p="0" yaw="0" axis_x="-0.7071" axis_y="-0.7071" axis_z="0" mesh_housing="model://omni4/meshes/omni_housing.stl" mesh_barrel="model://omni4/meshes/omni_barrel.stl"/>
+  <xacro:odm_visual_wheel name="wheel_front_right" x="${wheel_x}" y="-${wheel_y}" r="0" p="0" yaw="0" mesh_housing="model://omni4/meshes/omni_housing.stl" mesh_barrel="model://omni4/meshes/omni_barrel.stl"/>
+  <xacro:odm_visual_wheel name="wheel_rear_left" x="-${wheel_x}" y="${wheel_y}" r="0" p="0" yaw="0" mesh_housing="model://omni4/meshes/omni_housing.stl" mesh_barrel="model://omni4/meshes/omni_barrel.stl"/>
+  <xacro:odm_visual_wheel name="wheel_rear_right" x="-${wheel_x}" y="-${wheel_y}" r="0" p="0" yaw="0" mesh_housing="model://omni4/meshes/omni_housing.stl" mesh_barrel="model://omni4/meshes/omni_barrel.stl"/>
+<!-- まずはwheel_front_leftについてのみ考える -->
+<!-- 目標：車輪とモーターの接続部分が最初(-1,-1,0)方向(ベクトル)を向いて、(-1,-1,0)軸回転。 -->
+<!-- (r, p, yaw, axis_x, axis_y, axis_z) = (0, 0, 0, 0, 0, 1)のとき、接続部分が最初(0, 0, -1)方向を向いて、(0, 0, 1)軸回転 -->
+<!-- (r, p, yaw, axis_x, axis_y, axis_z) = (1.570796, 0, 0, 0, 0, 1)のとき、接続部分が最初(0, 0, 1)方向を向いて、(0, -1, 0)軸回転 -->
+<!-- (r, p, yaw, axis_x, axis_y, axis_z) = (0.785398, 0, 0, 0, 0, 1)のとき、接続部分が最初(0, 1, 0)方向を向いて、(0, -1, 1)軸回転 -->
+<!-- (r, p, yaw, axis_x, axis_y, axis_z) = (-0.785398, 0, -0.5, 0, 0, 1)のとき、接続部分が最初(-1, -1, 0)方向を向いて、(1, 1, 1)軸回転 -->
+<!-- (r, p, yaw, axis_x, axis_y, axis_z) = (1.5708, 0, -2.35619, 0, 0, 1)のとき、接続部分が最初(-1, -1, -1)方向を向いて、(-1, 1, 0)軸回転 -->
+  <!-- Create four wheels using meshes from sim2_lecture if available
   <xacro:odm_visual_wheel name="wheel_front_left" x="${wheel_x}" y="${wheel_y}" r="1.570796" p="0" yaw="0.7854" mesh_housing="model://omni4/meshes/omni_housing.stl" mesh_barrel="model://omni4/meshes/omni_barrel.stl"/>
   <xacro:odm_visual_wheel name="wheel_front_right" x="${wheel_x}" y="-${wheel_y}" r="1.570796" p="0" yaw="-0.7854" mesh_housing="model://omni4/meshes/omni_housing.stl" mesh_barrel="model://omni4/meshes/omni_barrel.stl"/>
   <xacro:odm_visual_wheel name="wheel_rear_left" x="-${wheel_x}" y="${wheel_y}" r="-1.570796" p="0" yaw="2.3562" mesh_housing="model://omni4/meshes/omni_housing.stl" mesh_barrel="model://omni4/meshes/omni_barrel.stl"/>
-  <xacro:odm_visual_wheel name="wheel_rear_right" x="-${wheel_x}" y="-${wheel_y}" r="-1.570796" p="0" yaw="-2.3562" mesh_housing="model://omni4/meshes/omni_housing.stl" mesh_barrel="model://omni4/meshes/omni_barrel.stl"/>
+  <xacro:odm_visual_wheel name="wheel_rear_right" x="-${wheel_x}" y="-${wheel_y}" r="-1.570796" p="0" yaw="-2.3562" mesh_housing="model://omni4/meshes/omni_housing.stl" mesh_barrel="model://omni4/meshes/omni_barrel.stl"/> -->
   <!-- ros2_control plugin config (keep velocity interfaces compatible with existing controllers) -->
   <ros2_control name="GazeboSystem" type="system">

Commit message: 色々実験

File: models/omni4/omni4.urdf (robot description, URDF)
Before this commit: robot omni4_robot, 5 links, 4 joints
Joints:
- joint wheel_front_left_joint: origin xyz=0.12 0.095 0.02 rpy=1.5708 0 -2.35619 -> xyz=0.12 0.095 0.02 rpy=0 -1.5708 -2.3561

File: urdf/omni4.urdf.xacro (robot description, xacro)
@@ -67,5 +67,5 @@
   </xacro:macro>
   <!-- Create four wheels using meshes from sim2_lecture if available -->
-  <xacro:odm_visual_wheel name="wheel_front_left" x="${wheel_x}" y="${wheel_y}" r="0" p="0" yaw="0" axis_x="-0.7071" axis_y="-0.7071" axis_z="0" mesh_housing="model://omni4/meshes/omni_housing.stl" mesh_barrel="model://omni4/meshes/omni_barrel.stl"/>
+  <xacro:odm_visual_wheel name="wheel_front_left" x="${wheel_x}" y="${wheel_y}" r="0" p="-1.5708" yaw="-2.3561" axis_x="0" axis_y="0" axis_z="1" mesh_housing="model://omni4/meshes/omni_housing.stl" mesh_barrel="model://omni4/meshes/omni_barrel.stl"/>
   <xacro:odm_visual_wheel name="wheel_front_right" x="${wheel_x}" y="-${wheel_y}" r="0" p="0" yaw="0" mesh_housing="model://omni4/meshes/omni_housing.stl" mesh_barrel="model://omni4/meshes/omni_barrel.stl"/>
   <xacro:odm_visual_wheel name="wheel_rear_left" x="-${wheel_x}" y="${wheel_y}" r="0" p="0" yaw="0" mesh_housing="model://omni4/meshes/omni_housing.stl" mesh_barrel="model://omni4/meshes/omni_barrel.stl"/>
@@ -78,4 +78,8 @@
 <!-- (r, p, yaw, axis_x, axis_y, axis_z) = (-0.785398, 0, -0.5, 0, 0, 1)のとき、接続部分が最初(-1, -1, 0)方向を向いて、(1, 1, 1)軸回転 -->
 <!-- (r, p, yaw, axis_x, axis_y, axis_z) = (1.5708, 0, -2.35619, 0, 0, 1)のとき、接続部分が最初(-1, -1, -1)方向を向いて、(-1, 1, 0)軸回転 -->
+<!-- r="0" p="1.5708" yaw="-2.35619" axis_x="-0.7071" axis_y="-0.7071" axis_z="0"のとき、接続部分が最初(1, -1, -1)方向を向いて、(-1, 1, 1)を軸に回転 -->
+<!-- r="0" p="1.5708" yaw="-2.3561" axis_x="0" axis_y="0" axis_z="1"のとき、接続部分が最初(1, -1, -1)方向を向いて、(-1, -1, 0)を軸に回転 -->
+<!-- r="0" p="0" yaw="-2.3561" axis_x="0" axis_y="0" axis_z="1"のとき、接続部分が最初(0, 0, -1)方向を向いて、(0, 0, 1)を軸に回転 -->
+<!-- r="0" p="-1.5708" yaw="-2.3561" axis_x="0" axis_y="0" axis_z="1"のとき、接続部分が最初(-1, 1, -1)方向を向いて、(-1, -1, 0)を軸に回転 -->
   <!-- Create four wheels using meshes from sim2_lecture if available
   <xacro:odm_visual_wheel name="wheel_front_left" x="${wheel_x}" y="${wheel_y}" r="1.570796" p="0" yaw="0.7854" mesh_housing="model://omni4/meshes/omni_housing.stl" mesh_barrel="model://omni4/meshes/omni_barrel.stl"/>

Commit message: おむに回転軸が変〜

File: models/omni4/omni4.urdf (robot description, URDF)
Before this commit: robot omni4_robot, 5 links, 4 joints
Joints:
- joint wheel_front_left_joint: axis 0 0 1 -> 0.7071 0.7071 1; origin xyz=0.12 0.095 0.02 rpy=0 -1.5708 -2.3561 -> xyz=0.12 0.095 0.02 rpy=-0.7071 0 -0.5

File: urdf/omni4.urdf.xacro (robot description, xacro)
@@ -67,5 +67,5 @@
   </xacro:macro>
   <!-- Create four wheels using meshes from sim2_lecture if available -->
-  <xacro:odm_visual_wheel name="wheel_front_left" x="${wheel_x}" y="${wheel_y}" r="0" p="-1.5708" yaw="-2.35610" axis_x="0" axis_y="0" axis_z="1" mesh_housing="model://omni4/meshes/omni_housing.stl" mesh_barrel="model://omni4/meshes/omni_barrel.stl"/>
+  <xacro:odm_visual_wheel name="wheel_front_left" x="${wheel_x}" y="${wheel_y}" r="-0.7071" p="0" yaw="-0.5" axis_x="0.7071" axis_y="0.7071" axis_z="1" mesh_housing="model://omni4/meshes/omni_housing.stl" mesh_barrel="model://omni4/meshes/omni_barrel.stl"/>
   <xacro:odm_visual_wheel name="wheel_front_right" x="${wheel_x}" y="-${wheel_y}" r="0" p="0" yaw="0" mesh_housing="model://omni4/meshes/omni_housing.stl" mesh_barrel="model://omni4/meshes/omni_barrel.stl"/>
   <xacro:odm_visual_wheel name="wheel_rear_left" x="-${wheel_x}" y="${wheel_y}" r="0" p="0" yaw="0" mesh_housing="model://omni4/meshes/omni_housing.stl" mesh_barrel="model://omni4/meshes/omni_barrel.stl"/>
