Commit message: ネットのやつを忠実再現途中。launchえらー

File: models/omni4/omni4.urdf (robot description, URDF)
Before this commit: robot omni4_robot, 5 links, 4 joints
Joints:
- joint wheel_front_left_joint: axis 0.7071 0.7071 1 -> 0 0 1; origin xyz=0.12 0.095 0.02 rpy=-0.7071 0 -0.5 -> xyz=0.12 0.095 0.02 rpy=0.7853 0 0

File: urdf/omni4.urdf.xacro (robot description, xacro)
@@ -67,5 +67,34 @@
   </xacro:macro>
   <!-- Create four wheels using meshes from sim2_lecture if available -->
-  <xacro:odm_visual_wheel name="wheel_front_left" x="${wheel_x}" y="${wheel_y}" r="-0.7071" p="0" yaw="-0.5" axis_x="0.7071" axis_y="0.7071" axis_z="1" mesh_housing="model://omni4/meshes/omni_housing.stl" mesh_barrel="model://omni4/meshes/omni_barrel.stl"/>
+  <xacro:odm_visual_wheel name="wheel_front_left" x="${wheel_x}" y="${wheel_y}" r="0" p="1.5708" yaw="-2.35619" axis_x="0" axis_y="0" axis_z="1" mesh_housing="model://omni4/meshes/omni_housing.stl" mesh_barrel="model://omni4/meshes/omni_barrel.stl"/>
+    <link name="wheel_front_left_link">
+      <inertial>
+        <mass value="${wheel_mass}"/>
+        <inertia ixx="0.00001" ixy="0" ixz="0" iyy="0.00001" iyz="0" izz="0.00002"/>
+      </inertial>
+      <visual>
+        <origin xyz="0 0 0" rpy="0 0 0"/>
+        <geometry>
+          <mesh filename="model://omni4/meshes/omni_barrel.stl"/>
+        </geometry>
+      </visual>
+      <collision>
+        <origin xyz="0 0 0" rpy="0 0 0"/>
+        <geometry>
+          <mesh filename="model://omni4/meshes/omni_barrel.stl"/>
+        </geometry>
+      </collision>
+    </link>
+    <gazebo reference="wheel_front_left_link">
+      <material>Gazebo/Grey</material>
+    </gazebo>
+    <joint name="wheel_front_left_joint" type="continuous">
+      <parent link="base_link"/>
+      <child link="wheel_front_left_link"/>
+      <origin xyz="${wheel_x} ${wheel_y} 0.02" rpy="0 1.5708 -2.35619"/>
+      <axis xyz="0 0 1"/>
+      <limit effort="10" velocity="20"/>
+      <dynamics damping="0.0" friction="0.0"/>
+    </joint>
   <xacro:odm_visual_wheel name="wheel_front_right" x="${wheel_x}" y="-${wheel_y}" r="0" p="0" yaw="0" mesh_housing="model://omni4/meshes/omni_housing.stl" mesh_barrel="model://omni4/meshes/omni_barrel.stl"/>
   <xacro:odm_visual_wheel name="wheel_rear_left" x="-${wheel_x}" y="${wheel_y}" r="0" p="0" yaw="0" mesh_housing="model://omni4/meshes/omni_housing.stl" mesh_barrel="model://omni4/meshes/omni_barrel.stl"/>
@@ -78,8 +107,5 @@
 <!-- (r, p, yaw, axis_x, axis_y, axis_z) = (-0.785398, 0, -0.5, 0, 0, 1)のとき、接続部分が最初(-1, -1, 0)方向を向いて、(1, 1, 1)軸回転 -->
 <!-- (r, p, yaw, axis_x, axis_y, axis_z) = (1.5708, 0, -2.35619, 0, 0, 1)のとき、接続部分が最初(-1, -1, -1)方向を向いて、(-1, 1, 0)軸回転 -->
-<!-- r="0" p="1.5708" yaw="-2.35619" axis_x="-0.7071" axis_y="-0.7071" axis_z="0"のとき、接続部分が最初(1, -1, -1)方向を向いて、(-1, 1, 1)を軸に回転 -->
-<!-- r="0" p="1.5708" yaw="-2.3561" axis_x="0" axis_y="0" axis_z="1"のとき、接続部分が最初(1, -1, -1)方向を向いて、(-1, -1, 0)を軸に回転 -->
-<!-- r="0" p="0" yaw="-2.3561" axis_x="0" axis_y="0" axis_z="1"のとき、接続部分が最初(0, 0, -1)方向を向いて、(0, 0, 1)を軸に回転 -->
-<!-- r="0" p="-1.5708" yaw="-2.3561" axis_x="0" axis_y="0" axis_z="1"のとき、接続部分が最初(-1, 1, -1)方向を向いて、(-1, -1, 0)を軸に回転 -->
+<!-- r="0" p="1.5708" yaw="-2.35619" axis_x="-0.7071" axis_y="-0.7071" axis_z="0"のとき、接続部分が最初(1, -1, -1)方向を向いて、(-1, 1, 1) -->
   <!-- Create four wheels using meshes from sim2_lecture if available
   <xacro:odm_visual_wheel name="wheel_front_left" x="${wheel_x}" y="${wheel_y}" r="1.570796" p="0" yaw="0.7854" mesh_housing="model://omni4/meshes/omni_housing.stl" mesh_barrel="model://omni4/meshes/omni_barrel.stl"/>
