Commit message: windousからarm_1のデータを持ってきて、.urdfに変換

File: models/arm_1/arm_1.urdf (robot description, URDF)
Before this commit: robot arm_1, 2 links, 1 joints
Links:
- link body_link: geometry collision mesh filename=meshes/entyu.stl scale=0.001 0.001 0.001; visual mesh filename=meshes/entyu.stl scale=0.001 0.001 0.001

File: urdf/arm_1.urdf.xacro (robot description, xacro)
@@ -1,4 +1,6 @@
 <?xml version="1.0"?>
 <robot xmlns:xacro="http://www.ros.org/wiki/xacro" name="arm_1">
+  <xacro:include filename="$(find gazebo_simulator)/models/omni_robot/omni_common.xacro"/>
+  <xacro:property name="model_scale" value="0.001"/>
   <link name="base_link"/>
   <joint name="body_joint" type="fixed">
@@ -10,5 +12,5 @@
     <visual>
       <geometry>
-        <mesh filename="meshes/entyu.stl" scale="1 1 1"/>
+        <mesh filename="meshes/entyu.stl" scale="${model_scale} ${model_scale} ${model_scale}"/>
       </geometry>
       <material name="gray"/>
@@ -16,5 +18,5 @@
     <collision>
       <geometry>
-        <mesh filename="meshes/entyu.stl" scale="1 1 1"/>
+        <mesh filename="meshes/entyu.stl" scale="${model_scale} ${model_scale} ${model_scale}"/>
       </geometry>
     </collision>

Commit message: gazeboでarmはスポーンはした

File: models/arm_1/arm_1.urdf (robot description, URDF)
Before this commit: robot arm_1, 2 links, 1 joints
Links:
- link arm_link_1_v2_2: geometry collision mesh filename=package://arm_1/meshes/arm_link_1_v2_2.stl scale=0.001 0.001 0.001; visual mesh filename=package://arm_1/meshes/arm_link_1_v2_2.stl scale=0.001 0.001 0.001
- link base_link: geometry collision mesh filename=package://arm_1/meshes/base_link.stl scale=0.001 0.001 0.001; visual mesh filename=package://arm_1/meshes/base_link.stl scale=0.001 0.001 0.001

File: models/arm_1/urdf/arm_1.xacro (robot description, xacro)
@@ -1,6 +1,6 @@
 <?xml version="1.0" ?>
 <robot name="arm_1" xmlns:xacro="http://www.ros.org/wiki/xacro">
-<xacro:include filename="$(find gazebo_simulator)/models/arm_1_description/urdf/materials.xacro" />
-<xacro:include filename="$(find gazebo_simulator)/models/arm_1_description/urdf/arm_1.trans" />
+<xacro:include filename="$(find gazebo_simulator)/models/arm_1/urdf/materials.xacro" />
+<xacro:include filename="$(find gazebo_simulator)/models/arm_1/urdf/arm_1.trans" />
 <link name="base_link">
   <inertial>
@@ -12,5 +12,5 @@
     <origin xyz="0 0 0" rpy="0 0 0"/>
     <geometry>
-      <mesh filename="package://arm_1_description/meshes/base_link.stl" scale="0.001 0.001 0.001"/>
+      <mesh filename="package://arm_1/meshes/base_link.stl" scale="0.001 0.001 0.001"/>
     </geometry>
     <material name="_"/>
@@ -19,5 +19,5 @@
     <origin xyz="0 0 0" rpy="0 0 0"/>
     <geometry>
-      <mesh filename="package://arm_1_description/meshes/base_link.stl" scale="0.001 0.001 0.001"/>
+      <mesh filename="package://arm_1/meshes/base_link.stl" scale="0.001 0.001 0.001"/>
     </geometry>
   </collision>
@@ -32,5 +32,5 @@
     <origin xyz="0.023999 0.007388 -0.116611" rpy="0 0 0"/>
     <geometry>
-      <mesh filename="package://arm_1_description/meshes/arm_link_1_v2_2.stl" scale="0.001 0.001 0.001"/>
+      <mesh filename="package://arm_1/meshes/arm_link_1_v2_2.stl" scale="0.001 0.001 0.001"/>
     </geometry>
     <material name="_"/>
@@ -39,5 +39,5 @@
     <origin xyz="0.023999 0.007388 -0.116611" rpy="0 0 0"/>
     <geometry>
-      <mesh filename="package://arm_1_description/meshes/arm_link_1_v2_2.stl" scale="0.001 0.001 0.001"/>
+      <mesh filename="package://arm_1/meshes/arm_link_1_v2_2.stl" scale="0.001 0.001 0.001"/>
     </geometry>
   </collision>
