Commit message: スポーンはした。うれしい。

File: models/arm_1/urdf/arm_1.xacro (robot description, xacro)
@@ -49,3 +49,29 @@
   <axis xyz="-0.0 0.0 -1.0"/>
 </joint>
+<!-- ros2_control plugin config (keep velocity interfaces compatible with existing controllers) -->
+<ros2_control name="GazeboSystem" type="system">
+  <hardware>
+    <plugin>gz_ros2_control/GazeboSimSystem</plugin>
+  </hardware>
+  <joint name="motor_1">
+    <command_interface name="velocity"/>
+    <state_interface name="position"/>
+    <state_interface name="velocity"/>
+  </joint>
+</ros2_control>
+<gazebo>
+  <plugin filename="libgz_ros2_control-system.so" name="gz_ros2_control::GazeboSimROS2ControlPlugin">
+    <parameters>$(find gazebo_simulator)/config/controller_omni_robot.yaml</parameters>
+  </plugin>
+</gazebo>
+<gazebo>
+  <plugin
+    filename="libgz-sim-pose-publisher-system.so"
+    name="gz::sim::systems::PosePublisher">
+    <publish_link_pose>true</publish_link_pose>
+    <publish_model_pose>true</publish_model_pose>
+    <use_pose_vector_msg>true</use_pose_vector_msg>
+    <update_frequency>50</update_frequency>
+  </plugin>
+</gazebo>
 </robot>

Commit message: モデル変更がしやすいように変更

File: models/arm_1/urdf/arm_1.xacro (robot description, xacro)
@@ -1,6 +1,7 @@
 <?xml version="1.0" ?>
 <robot name="arm_1" xmlns:xacro="http://www.ros.org/wiki/xacro">
-<xacro:include filename="$(find gazebo_simulator)/models/arm_1/urdf/materials.xacro" />
-<xacro:include filename="$(find gazebo_simulator)/models/arm_1/urdf/arm_1.trans" />
+<xacro:property name="robot_name" value="$(arg robot_name)"/>
+<xacro:include filename="$(find gazebo_simulator)/models/${robot_name}/urdf/materials.xacro" />
+<xacro:include filename="$(find gazebo_simulator)/models/${robot_name}/urdf/${robot_name}.trans" />
 <link name="base_link">
   <inertial>

File: models/arm_2/urdf/arm_2.xacro (robot description, xacro)
@@ -1,5 +1,5 @@
 <?xml version="1.0" ?>
 <robot name="arm_2" xmlns:xacro="http://www.ros.org/wiki/xacro">
-<xacro:property name="robot_name" value="arm_2"/>
+<xacro:property name="robot_name" value="$(arg robot_name)"/>
 <xacro:include filename="$(find gazebo_simulator)/models/${robot_name}/urdf/materials.xacro" />
 <xacro:include filename="$(find gazebo_simulator)/models/${robot_name}/urdf/${robot_name}.trans" />
