Commit message: おむにうごいたあああああ！！！

File: models/omni_robot/omni_robot.urdf (robot description, URDF)
Before this commit: robot omni_robot, 90 links, 89 joints
Joints:
- removed joint wheel_front_left_joint
- removed joint wheel_front_right_joint
- removed joint wheel_rear_left_joint
- removed joint wheel_rear_right_joint
- added joint wheel0_attach_joint: type fixed, parent base_link, child wheel0_attach_link, origin xyz=4.286263797015737e-18 0.07 0.019 rpy=0 0 1.5707963267948966
- added joint wheel1_attach_joint: type fixed, parent base_link, child wheel1_attach_link, origin xyz=-0.07 8.572527594031473e-18 0.019 rpy=0 0 3.141592653589793
- added joint wheel2_attach_joint: type fixed, parent base_link, child wheel2_attach_link, origin xyz=-1.285879139104721e-17 -0.07 0.019 rpy=0 0 4.71238898038469
- added joint wheel3_attach_joint: type fixed, parent base_link, child wheel3_attach_link, origin xyz=0.07 -1.7145055188062947e-17 0.019 rpy=0 0 6.283185307179586

File: urdf/omni_robot.urdf.xacro (robot description, xacro)
@@ -26,5 +26,5 @@
     </inertial>
   </link>
-  <joint name="wheel_front_left_joint" type="fixed">
+  <joint name="wheel0_attach_joint" type="fixed">
     <parent link="base_link"/>
     <child  link="wheel0_attach_link"/>
@@ -33,5 +33,5 @@
   <link name="wheel0_attach_link" />
   <xacro:omni_wheel_set prefix="wheel0" parent="wheel0_attach_link" />
-  <joint name="wheel_front_right_joint" type="fixed">
+  <joint name="wheel1_attach_joint" type="fixed">
     <parent link="base_link"/>
     <child  link="wheel1_attach_link"/>
@@ -40,5 +40,5 @@
   <link name="wheel1_attach_link" />
   <xacro:omni_wheel_set prefix="wheel1" parent="wheel1_attach_link" />
-  <joint name="wheel_rear_left_joint" type="fixed">
+  <joint name="wheel2_attach_joint" type="fixed">
     <parent link="base_link"/>
     <child  link="wheel2_attach_link"/>
@@ -47,5 +47,5 @@
   <link name="wheel2_attach_link" />
   <xacro:omni_wheel_set prefix="wheel2" parent="wheel2_attach_link" />
-  <joint name="wheel_rear_right_joint" type="fixed">
+  <joint name="wheel3_attach_joint" type="fixed">
     <parent link="base_link"/>
     <child  link="wheel3_attach_link"/>
@@ -59,20 +59,20 @@
       <plugin>gz_ros2_control/GazeboSimSystem</plugin>
     </hardware>
-    <joint name="wheel_front_left_joint">
+    <joint name="wheel0_motor_shaft_joint">
       <command_interface name="velocity"/>
       <state_interface name="position"/>
       <state_interface name="velocity"/>
     </joint>
-    <joint name="wheel_front_right_joint">
+    <joint name="wheel1_motor_shaft_joint">
       <command_interface name="velocity"/>
       <state_interface name="position"/>
       <state_interface name="velocity"/>
     </joint>
-    <joint name="wheel_rear_left_joint">
+    <joint name="wheel2_motor_shaft_joint">
       <command_interface name="velocity"/>
       <state_interface name="position"/>
       <state_interface name="velocity"/>
     </joint>
-    <joint name="wheel_rear_right_joint">
+    <joint name="wheel3_motor_shaft_joint">
       <command_interface name="velocity"/>
       <state_interface name="position"/>
@@ -82,5 +82,5 @@
   <gazebo>
     <plugin filename="libgz_ros2_control-system.so" name="gz_ros2_control::GazeboSimROS2ControlPlugin">
-      <parameters>$(find gazebo_simulator)/config/controller_omni4.yaml</parameters>
+      <parameters>$(find gazebo_simulator)/config/controller_omni_robot.yaml</parameters>
     </plugin>
   </gazebo>

Commit message: ros2 topic echo /tfで各モーターの情報getだぜ！

File: models/omni_robot/omni_robot.urdf (robot description, URDF)
Before this commit: robot omni_robot, 90 links, 89 joints
Joints:
- joint wheel0_attach_joint: origin xyz=4.286263797015737e-18 0.07 0.019 rpy=0 0 1.5707963267948966 -> xyz=0.04949747468305833 0.049497474683058325 0.019 rpy=0 0 0.7853981633974483
- joint wheel1_attach_joint: origin xyz=-0.07 8.572527594031473e-18 0.019 rpy=0 0 3.141592653589793 -> xyz=-0.049497474683058325 0.04949747468305833 0.019 rpy=0 0 2.356194490192345
- joint wheel2_attach_joint: origin xyz=-1.285879139104721e-17 -0.07 0.019 rpy=0 0 4.71238898038469 -> xyz=-0.049497474683058346 -0.049497474683058325 0.019 rpy=0 0 3.9269908169872414
- joint wheel3_attach_joint: origin xyz=0.07 -1.7145055188062947e-17 0.019 rpy=0 0 6.283185307179586 -> xyz=0.04949747468305832 -0.049497474683058346 0.019 rpy=0 0 5.497787143782138

File: urdf/omni_robot.urdf.xacro (robot description, xacro)
@@ -29,5 +29,5 @@
     <parent link="base_link"/>
     <child  link="wheel0_attach_link"/>
-    <origin xyz="${0.07*cos(radians(90))} ${0.07*sin(radians(90))} 0.019" rpy="0 0 ${radians(90)}"/>
+    <origin xyz="${0.07*cos(radians(45))} ${0.07*sin(radians(45))} 0.019" rpy="0 0 ${radians(45)}"/>
   </joint>
   <link name="wheel0_attach_link" />
@@ -36,5 +36,5 @@
     <parent link="base_link"/>
     <child  link="wheel1_attach_link"/>
-    <origin xyz="${0.07*cos(radians(180))} ${0.07*sin(radians(180))} 0.019" rpy="0 0 ${radians(180)}"/>
+    <origin xyz="${0.07*cos(radians(135))} ${0.07*sin(radians(135))} 0.019" rpy="0 0 ${radians(135)}"/>
   </joint>
   <link name="wheel1_attach_link" />
@@ -43,5 +43,5 @@
     <parent link="base_link"/>
     <child  link="wheel2_attach_link"/>
-    <origin xyz="${0.07*cos(radians(270))} ${0.07*sin(radians(270))} 0.019" rpy="0 0 ${radians(270)}"/>
+    <origin xyz="${0.07*cos(radians(225))} ${0.07*sin(radians(225))} 0.019" rpy="0 0 ${radians(225)}"/>
   </joint>
   <link name="wheel2_attach_link" />
@@ -50,5 +50,5 @@
     <parent link="base_link"/>
     <child  link="wheel3_attach_link"/>
-    <origin xyz="${0.07*cos(radians(360))} ${0.07*sin(radians(360))} 0.019" rpy="0 0 ${radians(360)}"/>
+    <origin xyz="${0.07*cos(radians(315))} ${0.07*sin(radians(315))} 0.019" rpy="0 0 ${radians(315)}"/>
   </joint>
   <link name="wheel3_attach_link" />
@@ -85,3 +85,13 @@
     </plugin>
   </gazebo>
+  <gazebo>
+    <plugin
+      filename="libgz-sim-pose-publisher-system.so"
+      name="gz::sim::systems::PosePublisher">
+      <publish_link_pose>false</publish_link_pose>
+      <publish_model_pose>true</publish_model_pose>
+      <use_pose_vector_msg>true</use_pose_vector_msg>
+      <update_frequency>50</update_frequency>
+    </plugin>
+  </gazebo>
 </robot>

Commit message: 姿勢補正しながらおむに動かせた！

File: models/omni_robot/omni_robot.urdf (robot description, URDF)
Before this commit: robot omni_robot, 90 links, 89 joints
Joints:
- joint wheel0_attach_joint: origin xyz=0.04949747468305833 0.049497474683058325 0.019 rpy=0 0 0.7853981633974483 -> xyz=0.04949747468305833 -0.049497474683058325 0.019 rpy=0 0 -0.7853981633974483
- joint wheel1_attach_joint: origin xyz=-0.049497474683058325 0.04949747468305833 0.019 rpy=0 0 2.356194490192345 -> xyz=0.04949747468305833 0.049497474683058325 0.019 rpy=0 0 0.7853981633974483
- joint wheel2_attach_joint: origin xyz=-0.049497474683058346 -0.049497474683058325 0.019 rpy=0 0 3.9269908169872414 -> xyz=-0.049497474683058325 0.04949747468305833 0.019 rpy=0 0 2.356194490192345
- joint wheel3_attach_joint: origin xyz=0.04949747468305832 -0.049497474683058346 0.019 rpy=0 0 5.497787143782138 -> xyz=-0.049497474683058346 -0.049497474683058325 0.019 rpy=0 0 3.9269908169872414

File: urdf/omni_robot.urdf.xacro (robot description, xacro)
@@ -3,4 +3,9 @@
   <xacro:include filename="$(find gazebo_simulator)/models/omni_robot/omni_common.xacro"/>
   <xacro:include filename="$(find gazebo_simulator)/models/omni_robot/omni_wheel.xacro"/>
+  <!-- per-wheel mounting angles (degrees) - change these to reposition wheels easily -->
+  <xacro:property name="wheel0_angle_deg" value="-45"/>
+  <xacro:property name="wheel1_angle_deg" value="45"/>
+  <xacro:property name="wheel2_angle_deg" value="135"/>
+  <xacro:property name="wheel3_angle_deg" value="225"/>
   <link name="base_link"/>
   <joint name="body_joint" type="fixed">
@@ -29,5 +34,5 @@
     <parent link="base_link"/>
     <child  link="wheel0_attach_link"/>
-    <origin xyz="${0.07*cos(radians(45))} ${0.07*sin(radians(45))} 0.019" rpy="0 0 ${radians(45)}"/>
+    <origin xyz="${0.07*cos(radians(wheel0_angle_deg))} ${0.07*sin(radians(wheel0_angle_deg))} 0.019" rpy="0 0 ${radians(wheel0_angle_deg)}"/>
   </joint>
   <link name="wheel0_attach_link" />
@@ -36,5 +41,5 @@
     <parent link="base_link"/>
     <child  link="wheel1_attach_link"/>
-    <origin xyz="${0.07*cos(radians(135))} ${0.07*sin(radians(135))} 0.019" rpy="0 0 ${radians(135)}"/>
+    <origin xyz="${0.07*cos(radians(wheel1_angle_deg))} ${0.07*sin(radians(wheel1_angle_deg))} 0.019" rpy="0 0 ${radians(wheel1_angle_deg)}"/>
   </joint>
   <link name="wheel1_attach_link" />
@@ -43,5 +48,5 @@
     <parent link="base_link"/>
     <child  link="wheel2_attach_link"/>
-    <origin xyz="${0.07*cos(radians(225))} ${0.07*sin(radians(225))} 0.019" rpy="0 0 ${radians(225)}"/>
+    <origin xyz="${0.07*cos(radians(wheel2_angle_deg))} ${0.07*sin(radians(wheel2_angle_deg))} 0.019" rpy="0 0 ${radians(wheel2_angle_deg)}"/>
   </joint>
   <link name="wheel2_attach_link" />
@@ -50,5 +55,5 @@
     <parent link="base_link"/>
     <child  link="wheel3_attach_link"/>
-    <origin xyz="${0.07*cos(radians(315))} ${0.07*sin(radians(315))} 0.019" rpy="0 0 ${radians(315)}"/>
+    <origin xyz="${0.07*cos(radians(wheel3_angle_deg))} ${0.07*sin(radians(wheel3_angle_deg))} 0.019" rpy="0 0 ${radians(wheel3_angle_deg)}"/>
   </joint>
   <link name="wheel3_attach_link" />

Commit message: twistの向きとgazeboで進む方向を一致

File: models/omni_robot/omni_robot.urdf (robot description, URDF)
Before this commit: robot omni_robot, 90 links, 89 joints
Joints:
- joint body_joint: origin xyz=0 0 0.05 rpy=0 0 0 -> xyz=0 0 0.05 rpy=0 0 1.5707963267948966
- joint wheel0_attach_joint: origin xyz=0.04949747468305833 -0.049497474683058325 0.019 rpy=0 0 -0.7853981633974483 -> xyz=0.04949747468305833 0.049497474683058325 0.019 rpy=0 0 0.7853981633974483
- joint wheel1_attach_joint: origin xyz=0.04949747468305833 0.049497474683058325 0.019 rpy=0 0 0.7853981633974483 -> xyz=-0.049497474683058325 0.04949747468305833 0.019 rpy=0 0 2.356194490192345
- joint wheel2_attach_joint: origin xyz=-0.049497474683058325 0.04949747468305833 0.019 rpy=0 0 2.356194490192345 -> xyz=-0.049497474683058346 -0.049497474683058325 0.019 rpy=0 0 3.9269908169872414
- joint wheel3_attach_joint: origin xyz=-0.049497474683058346 -0.049497474683058325 0.019 rpy=0 0 3.9269908169872414 -> xyz=0.04949747468305832 -0.049497474683058346 0.019 rpy=0 0 5.497787143782138

File: urdf/omni_robot.urdf.xacro (robot description, xacro)
@@ -4,13 +4,13 @@
   <xacro:include filename="$(find gazebo_simulator)/models/omni_robot/omni_wheel.xacro"/>
   <!-- per-wheel mounting angles (degrees) - change these to reposition wheels easily -->
-  <xacro:property name="wheel0_angle_deg" value="-45"/>
-  <xacro:property name="wheel1_angle_deg" value="45"/>
-  <xacro:property name="wheel2_angle_deg" value="135"/>
-  <xacro:property name="wheel3_angle_deg" value="225"/>
+  <xacro:property name="wheel0_angle_deg" value="45"/>
+  <xacro:property name="wheel1_angle_deg" value="135"/>
+  <xacro:property name="wheel2_angle_deg" value="225"/>
+  <xacro:property name="wheel3_angle_deg" value="315"/>
   <link name="base_link"/>
   <joint name="body_joint" type="fixed">
     <parent link="base_link"/>
     <child  link="body_link"/>
-    <origin xyz="0 0 0.05" rpy="0 0 0"/>
+    <origin xyz="0 0 0.05" rpy="0 0 ${radians(90)}"/>
   </joint>
   <link name="body_link">

Commit message: lidarのレーザー光をgazeboに可視化

File: models/omni_robot/omni_robot.urdf (robot description, URDF)
Before this commit: robot omni_robot, 90 links, 89 joints
Links:
- added link lidar_link, mass 0.05; collision cylinder length=0.035 radius=0.025; visual cylinder length=0.035 radius=0.025
Joints:
- added joint lidar_joint: type fixed, parent base_link, child lidar_link, origin xyz=0 0 0.075 rpy=0 0 0

File: models/omni_robot/urdf/omni_robot.xacro (robot description, xacro)
@@ -3,4 +3,5 @@
   <xacro:include filename="$(find gazebo_simulator)/models/omni_robot/omni_common.xacro"/>
   <xacro:include filename="$(find gazebo_simulator)/models/omni_robot/omni_wheel.xacro"/>
+  <xacro:include filename="$(find gazebo_simulator)/models/omni_robot/lidar.xacro"/>
   <!-- per-wheel mounting angles (degrees) - change these to reposition wheels easily -->
   <xacro:property name="wheel0_angle_deg" value="45"/>
@@ -31,4 +32,11 @@
     </inertial>
   </link>
+  <xacro:lidar_macro
+    prefix="lidar"
+    parent="base_link"
+    xyz="0 0 0.075"
+    rpy="0 0 0"
+    angle_min="${-pi}"
+    angle_max="${pi}"/>
   <joint name="wheel0_attach_joint" type="fixed">
     <parent link="base_link"/>
