Commit message: omni_robotサイズ変更。半径を変えやすくした

File: models/omni_robot/omni_robot.urdf (robot description, URDF)
Before this commit: robot omni_robot, 91 links, 90 joints
Links:
- link body_link: geometry collision box size=0.60 0.60 0.02; visual box size=0.60 0.60 0.02

File: models/omni_robot/urdf/omni_robot.xacro (robot description, xacro)
@@ -9,4 +9,5 @@
   <xacro:property name="wheel2_angle_deg" value="225"/>
   <xacro:property name="wheel3_angle_deg" value="315"/>
+  <xacro:property name="wheel_mount_radius" value="0.07"/>
   <link name="base_link"/>
   <joint name="body_joint" type="fixed">
@@ -18,5 +19,5 @@
     <visual>
       <geometry>
-        <box size="0.14 0.08 0.02" />
+        <box size="0.60 0.60 0.02" />
       </geometry>
       <material name="gray"/>
@@ -24,5 +25,5 @@
     <collision>
       <geometry>
-        <box size="0.14 0.08 0.02" />
+        <box size="0.60 0.60 0.02" />
       </geometry>
     </collision>
@@ -42,5 +43,9 @@
     <parent link="base_link"/>
     <child  link="wheel0_attach_link"/>
-    <origin xyz="${0.07*cos(radians(wheel0_angle_deg))} ${0.07*sin(radians(wheel0_angle_deg))} 0.019" rpy="0 0 ${radians(wheel0_angle_deg)}"/>
+    <origin
+      xyz="${wheel_mount_radius*cos(radians(wheel0_angle_deg))}
+          ${wheel_mount_radius*sin(radians(wheel0_angle_deg))}
+          0.019"
+      rpy="0 0 ${radians(wheel0_angle_deg)}"/>
   </joint>
   <link name="wheel0_attach_link" />
@@ -49,5 +54,9 @@
     <parent link="base_link"/>
     <child  link="wheel1_attach_link"/>
-    <origin xyz="${0.07*cos(radians(wheel1_angle_deg))} ${0.07*sin(radians(wheel1_angle_deg))} 0.019" rpy="0 0 ${radians(wheel1_angle_deg)}"/>
+    <origin
+      xyz="${wheel_mount_radius*cos(radians(wheel1_angle_deg))}
+          ${wheel_mount_radius*sin(radians(wheel1_angle_deg))}
+          0.019"
+      rpy="0 0 ${radians(wheel1_angle_deg)}"/>
   </joint>
   <link name="wheel1_attach_link" />
@@ -56,5 +65,9 @@
     <parent link="base_link"/>
     <child  link="wheel2_attach_link"/>
-    <origin xyz="${0.07*cos(radians(wheel2_angle_deg))} ${0.07*sin(radians(wheel2_angle_deg))} 0.019" rpy="0 0 ${radians(wheel2_angle_deg)}"/>
+    <origin
+      xyz="${wheel_mount_radius*cos(radians(wheel2_angle_deg))}
+          ${wheel_mount_radius*sin(radians(wheel2_angle_deg))}
+          0.019"
+      rpy="0 0 ${radians(wheel2_angle_deg)}"/>
   </joint>
   <link name="wheel2_attach_link" />
@@ -63,5 +76,9 @@
     <parent link="base_link"/>
     <child  link="wheel3_attach_link"/>
-    <origin xyz="${0.07*cos(radians(wheel3_angle_deg))} ${0.07*sin(radians(wheel3_angle_deg))} 0.019" rpy="0 0 ${radians(wheel3_angle_deg)}"/>
+    <origin
+  xyz="${wheel_mount_radius*cos(radians(wheel3_angle_deg))}
+       ${wheel_mount_radius*sin(radians(wheel3_angle_deg))}
+       0.019"
+  rpy="0 0 ${radians(wheel3_angle_deg)}"/>
   </joint>
   <link name="wheel3_attach_link" />

Commit message: 半径を変更したり

File: models/omni_robot/omni_robot.urdf (robot description, URDF)
Before this commit: robot omni_robot, 91 links, 90 joints
Joints:
- joint wheel0_attach_joint: origin xyz=0.04949747468305833 0.049497474683058325 0.019 rpy=0 0 0.7853981633974483 -> xyz=0.14142135623730953           0.1414213562373095           0.019 rpy=0 0 0.7853981633974483
- joint wheel1_attach_joint: origin xyz=-0.049497474683058325 0.04949747468305833 0.019 rpy=0 0 2.356194490192345 -> xyz=-0.1414213562373095           0.14142135623730953           0.019 rpy=0 0 2.356194490192345
- joint wheel2_attach_joint: origin xyz=-0.049497474683058346 -0.049497474683058325 0.019 rpy=0 0 3.9269908169872414 -> xyz=-0.14142135623730953           -0.1414213562373095           0.019 rpy=0 0 3.9269908169872414
- joint wheel3_attach_joint: origin xyz=0.04949747468305832 -0.049497474683058346 0.019 rpy=0 0 5.497787143782138 -> xyz=0.14142135623730948        -0.14142135623730953        0.019 rpy=0 0 5.497787143782138

File: models/omni_robot/urdf/omni_robot.xacro (robot description, xacro)
@@ -9,5 +9,5 @@
   <xacro:property name="wheel2_angle_deg" value="225"/>
   <xacro:property name="wheel3_angle_deg" value="315"/>
-  <xacro:property name="wheel_mount_radius" value="0.07"/>
+  <xacro:property name="wheel_mount_radius" value="0.2"/>
   <link name="base_link"/>
   <joint name="body_joint" type="fixed">

Commit message: おむにと車体でっかくなった。正常に動いた！

File: models/omni_robot/omni_robot.urdf (robot description, URDF)
Before this commit: robot omni_robot, 91 links, 90 joints
Links:
- link wheel0_barrel_1_link: geometry collision mesh filename=model://omni_robot/meshes/omni_barrel100.stl; visual mesh filename=model://omni_robot/meshes/omni_barrel100.stl
- link wheel0_barrel_2_link: geometry collision mesh filename=model://omni_robot/meshes/omni_barrel100.stl; visual mesh filename=model://omni_robot/meshes/omni_barrel100.stl
- link wheel0_barrel_3_link: geometry collision mesh filename=model://omni_robot/meshes/omni_barrel100.stl; visual mesh filename=model://omni_robot/meshes/omni_barrel100.stl
- link wheel0_barrel_4_link: geometry collision mesh filename=model://omni_robot/meshes/omni_barrel100.stl; visual mesh filename=model://omni_robot/meshes/omni_barrel100.stl
- link wheel0_barrel_5_link: geometry collision mesh filename=model://omni_robot/meshes/omni_barrel100.stl; visual mesh filename=model://omni_robot/meshes/omni_barrel100.stl
- link wheel0_barrel_6_link: geometry collision mesh filename=model://omni_robot/meshes/omni_barrel100.stl; visual mesh filename=model://omni_robot/meshes/omni_barrel100.stl
- link wheel0_barrel_7_link: geometry collision mesh filename=model://omni_robot/meshes/omni_barrel100.stl; visual mesh filename=model://omni_robot/meshes/omni_barrel100.stl
- link wheel0_barrel_8_link: geometry collision mesh filename=model://omni_robot/meshes/omni_barrel100.stl; visual mesh filename=model://omni_robot/meshes/omni_barrel100.stl
- link wheel0_housing_link: geometry visual mesh filename=model://omni_robot/meshes/omni_housing100.stl
- link wheel1_barrel_1_link: geometry collision mesh filename=model://omni_robot/meshes/omni_barrel100.stl; visual mesh filename=model://omni_robot/meshes/omni_barrel100.stl
- link wheel1_barrel_2_link: geometry collision mesh filename=model://omni_robot/meshes/omni_barrel100.stl; visual mesh filename=model://omni_robot/meshes/omni_barrel100.stl
- link wheel1_barrel_3_link: geometry collision mesh filename=model://omni_robot/meshes/omni_barrel100.stl; visual mesh filename=model://omni_robot/meshes/omni_barrel100.stl
- link wheel1_barrel_4_link: geometry collision mesh filename=model://omni_robot/meshes/omni_barrel100.stl; visual mesh filename=model://omni_robot/meshes/omni_barrel100.stl
- link wheel1_barrel_5_link: geometry collision mesh filename=model://omni_robot/meshes/omni_barrel100.stl; visual mesh filename=model://omni_robot/meshes/omni_barrel100.stl
- link wheel1_barrel_6_link: geometry collision mesh filename=model://omni_robot/meshes/omni_barrel100.stl; visual mesh filename=model://omni_robot/meshes/omni_barrel100.stl
- link wheel1_barrel_7_link: geometry collision mesh filename=model://omni_robot/meshes/omni_barrel100.stl; visual mesh filename=model://omni_robot/meshes/omni_barrel100.stl
- link wheel1_barrel_8_link: geometry collision mesh filename=model://omni_robot/meshes/omni_barrel100.stl; visual mesh filename=model://omni_robot/meshes/omni_barrel100.stl
- link wheel1_housing_link: geometry visual mesh filename=model://omni_robot/meshes/omni_housing100.stl
- link wheel2_barrel_1_link: geometry collision mesh filename=model://omni_robot/meshes/omni_barrel100.stl; visual mesh filename=model://omni_robot/meshes/omni_barrel100.stl
- link wheel2_barrel_2_link: geometry collision mesh filename=model://omni_robot/meshes/omni_barrel100.stl; visual mesh filename=model://omni_robot/meshes/omni_barrel100.stl
- link wheel2_barrel_3_link: geometry collision mesh filename=model://omni_robot/meshes/omni_barrel100.stl; visual mesh filename=model://omni_robot/meshes/omni_barrel100.stl
- link wheel2_barrel_4_link: geometry collision mesh filename=model://omni_robot/meshes/omni_barrel100.stl; visual mesh filename=model://omni_robot/meshes/omni_barrel100.stl
- link wheel2_barrel_5_link: geometry collision mesh filename=model://omni_robot/meshes/omni_barrel100.stl; visual mesh filename=model://omni_robot/meshes/omni_barrel100.stl
- link wheel2_barrel_6_link: geometry collision mesh filename=model://omni_robot/meshes/omni_barrel100.stl; visual mesh filename=model://omni_robot/meshes/omni_barrel100.stl
- link wheel2_barrel_7_link: geometry collision mesh filename=model://omni_robot/meshes/omni_barrel100.stl; visual mesh filename=model://omni_robot/meshes/omni_barrel100.stl
- link wheel2_barrel_8_link: geometry collision mesh filename=model://omni_robot/meshes/omni_barrel100.stl; visual mesh filename=model://omni_robot/meshes/omni_barrel100.stl
- link wheel2_housing_link: geometry visual mesh filename=model://omni_robot/meshes/omni_housing100.stl
- link wheel3_barrel_1_link: geometry collision mesh filename=model://omni_robot/meshes/omni_barrel100.stl; visual mesh filename=model://omni_robot/meshes/omni_barrel100.stl
- link wheel3_barrel_2_link: geometry collision mesh filename=model://omni_robot/meshes/omni_barrel100.stl; visual mesh filename=model://omni_robot/meshes/omni_barrel100.stl
- link wheel3_barrel_3_link: geometry collision mesh filename=model://omni_robot/meshes/omni_barrel100.stl; visual mesh filename=model://omni_robot/meshes/omni_barrel100.stl
- link wheel3_barrel_4_link: geometry collision mesh filename=model://omni_robot/meshes/omni_barrel100.stl; visual mesh filename=model://omni_robot/meshes/omni_barrel100.stl
- link wheel3_barrel_5_link: geometry collision mesh filename=model://omni_robot/meshes/omni_barrel100.stl; visual mesh filename=model://omni_robot/meshes/omni_barrel100.stl
- link wheel3_barrel_6_link: geometry collision mesh filename=model://omni_robot/meshes/omni_barrel100.stl; visual mesh filename=model://omni_robot/meshes/omni_barrel100.stl
- link wheel3_barrel_7_link: geometry collision mesh filename=model://omni_robot/meshes/omni_barrel100.stl; visual mesh filename=model://omni_robot/meshes/omni_barrel100.stl
- link wheel3_barrel_8_link: geometry collision mesh filename=model://omni_robot/meshes/omni_barrel100.stl; visual mesh filename=model://omni_robot/meshes/omni_barrel100.stl
- link wheel3_housing_link: geometry visual mesh filename=model://omni_robot/meshes/omni_housing100.stl
Joints:
- joint wheel0_attach_joint: origin xyz=0.14142135623730953           0.1414213562373095           0.019 rpy=0 0 0.7853981633974483 -> xyz=0.21213203435596426           0.21213203435596423           -0.04 rpy=0 0 0.7853981633974483
- joint wheel0_barrel_1_joint: origin xyz=0.014 0.0 0.006 rpy=1.5707963267948966 0 0 -> xyz=0.036842105 0.0 0.015789474 rpy=1.5707963267948966 0 0
- joint wheel0_barrel_2_joint: origin xyz=8.572527594031473e-19 0.014 0.006 rpy=1.5707963267948966 0 1.5707963267948966 -> xyz=2.2559282981050347e-18 0.036842105 0.015789474 rpy=1.5707963267948966 0 1.5707963267948966
- joint wheel0_barrel_3_joint: origin xyz=-0.014 1.7145055188062945e-18 0.006 rpy=1.5707963267948966 0 3.141592653589793 -> xyz=-0.036842105 4.5118565962100695e-18 0.015789474 rpy=1.5707963267948966 0 3.141592653589793
- joint wheel0_barrel_4_joint: origin xyz=8.572527594031473e-19 -0.014 0.006 rpy=1.5707963267948966 0 -1.5707963267948966 -> xyz=2.2559282981050347e-18 -0.036842105 0.015789474 rpy=1.5707963267948966 0 -1.5707963267948966
- joint wheel0_barrel_5_joint: origin xyz=0.014 0.0 0.006 rpy=1.5707963267948966 0 0 -> xyz=0.036842105 0.0 0.015789474 rpy=1.5707963267948966 0 0
- joint wheel0_barrel_6_joint: origin xyz=8.572527594031473e-19 0.014 0.006 rpy=1.5707963267948966 0 1.5707963267948966 -> xyz=2.2559282981050347e-18 0.036842105 0.015789474 rpy=1.5707963267948966 0 1.5707963267948966
- joint wheel0_barrel_7_joint: origin xyz=-0.014 1.7145055188062945e-18 0.006 rpy=1.5707963267948966 0 3.141592653589793 -> xyz=-0.036842105 4.5118565962100695e-18 0.015789474 rpy=1.5707963267948966 0 3.141592653589793
- joint wheel0_barrel_8_joint: origin xyz=8.572527594031473e-19 -0.014 0.006 rpy=1.5707963267948966 0 -1.5707963267948966 -> xyz=2.2559282981050347e-18 -0.036842105 0.015789474 rpy=1.5707963267948966 0 -1.5707963267948966
- joint wheel1_attach_joint: origin xyz=-0.1414213562373095           0.14142135623730953           0.019 rpy=0 0 2.356194490192345 -> xyz=-0.21213203435596423           0.21213203435596426           -0.04 rpy=0 0 2.356194490192345
- joint wheel1_barrel_1_joint: origin xyz=0.014 0.0 0.006 rpy=1.5707963267948966 0 0 -> xyz=0.036842105 0.0 0.015789474 rpy=1.5707963267948966 0 0
- joint wheel1_barrel_2_joint: origin xyz=8.572527594031473e-19 0.014 0.006 rpy=1.5707963267948966 0 1.5707963267948966 -> xyz=2.2559282981050347e-18 0.036842105 0.015789474 rpy=1.5707963267948966 0 1.5707963267948966
- joint wheel1_barrel_3_joint: origin xyz=-0.014 1.7145055188062945e-18 0.006 rpy=1.5707963267948966 0 3.141592653589793 -> xyz=-0.036842105 4.5118565962100695e-18 0.015789474 rpy=1.5707963267948966 0 3.141592653589793
- joint wheel1_barrel_4_joint: origin xyz=8.572527594031473e-19 -0.014 0.006 rpy=1.5707963267948966 0 -1.5707963267948966 -> xyz=2.2559282981050347e-18 -0.036842105 0.015789474 rpy=1.5707963267948966 0 -1.5707963267948966
- joint wheel1_barrel_5_joint: origin xyz=0.014 0.0 0.006 rpy=1.5707963267948966 0 0 -> xyz=0.036842105 0.0 0.015789474 rpy=1.5707963267948966 0 0
- joint wheel1_barrel_6_joint: origin xyz=8.572527594031473e-19 0.014 0.006 rpy=1.5707963267948966 0 1.5707963267948966 -> xyz=2.2559282981050347e-18 0.036842105 0.015789474 rpy=1.5707963267948966 0 1.5707963267948966
- joint wheel1_barrel_7_joint: origin xyz=-0.014 1.7145055188062945e-18 0.006 rpy=1.5707963267948966 0 3.141592653589793 -> xyz=-0.036842105 4.5118565962100695e-18 0.015789474 rpy=1.5707963267948966 0 3.141592653589793
- joint wheel1_barrel_8_joint: origin xyz=8.572527594031473e-19 -0.014 0.006 rpy=1.5707963267948966 0 -1.5707963267948966 -> xyz=2.2559282981050347e-18 -0.036842105 0.015789474 rpy=1.5707963267948966 0 -1.5707963267948966
- joint wheel2_attach_joint: origin xyz=-0.14142135623730953           -0.1414213562373095           0.019 rpy=0 0 3.9269908169872414 -> xyz=-0.2121320343559643           -0.21213203435596423           -0.04 rpy=0 0 3.9269908169872414
- joint wheel2_barrel_1_joint: origin xyz=0.014 0.0 0.006 rpy=1.5707963267948966 0 0 -> xyz=0.036842105 0.0 0.015789474 rpy=1.5707963267948966 0 0
- joint wheel2_barrel_2_joint: origin xyz=8.572527594031473e-19 0.014 0.006 rpy=1.5707963267948966 0 1.5707963267948966 -> xyz=2.2559282981050347e-18 0.036842105 0.015789474 rpy=1.5707963267948966 0 1.5707963267948966
- joint wheel2_barrel_3_joint: origin xyz=-0.014 1.7145055188062945e-18 0.006 rpy=1.5707963267948966 0 3.141592653589793 -> xyz=-0.036842105 4.5118565962100695e-18 0.015789474 rpy=1.5707963267948966 0 3.141592653589793
- joint wheel2_barrel_4_joint: origin xyz=8.572527594031473e-19 -0.014 0.006 rpy=1.5707963267948966 0 -1.5707963267948966 -> xyz=2.2559282981050347e-18 -0.036842105 0.015789474 rpy=1.5707963267948966 0 -1.5707963267948966
- joint wheel2_barrel_5_joint: origin xyz=0.014 0.0 0.006 rpy=1.5707963267948966 0 0 -> xyz=0.036842105 0.0 0.015789474 rpy=1.5707963267948966 0 0
- joint wheel2_barrel_6_joint: origin xyz=8.572527594031473e-19 0.014 0.006 rpy=1.5707963267948966 0 1.5707963267948966 -> xyz=2.2559282981050347e-18 0.036842105 0.015789474 rpy=1.5707963267948966 0 1.5707963267948966
- joint wheel2_barrel_7_joint: origin xyz=-0.014 1.7145055188062945e-18 0.006 rpy=1.5707963267948966 0 3.141592653589793 -> xyz=-0.036842105 4.5118565962100695e-18 0.015789474 rpy=1.5707963267948966 0 3.141592653589793
- joint wheel2_barrel_8_joint: origin xyz=8.572527594031473e-19 -0.014 0.006 rpy=1.5707963267948966 0 -1.5707963267948966 -> xyz=2.2559282981050347e-18 -0.036842105 0.015789474 rpy=1.5707963267948966 0 -1.5707963267948966
- joint wheel3_attach_joint: origin xyz=0.14142135623730948        -0.14142135623730953        0.019 rpy=0 0 5.497787143782138 -> xyz=0.2121320343559642        -0.2121320343559643        -0.04 rpy=0 0 5.497787143782138
- joint wheel3_barrel_1_joint: origin xyz=0.014 0.0 0.006 rpy=1.5707963267948966 0 0 -> xyz=0.036842105 0.0 0.015789474 rpy=1.5707963267948966 0 0
- joint wheel3_barrel_2_joint: origin xyz=8.572527594031473e-19 0.014 0.006 rpy=1.5707963267948966 0 1.5707963267948966 -> xyz=2.2559282981050347e-18 0.036842105 0.015789474 rpy=1.5707963267948966 0 1.5707963267948966
- joint wheel3_barrel_3_joint: origin xyz=-0.014 1.7145055188062945e-18 0.006 rpy=1.5707963267948966 0 3.141592653589793 -> xyz=-0.036842105 4.5118565962100695e-18 0.015789474 rpy=1.5707963267948966 0 3.141592653589793
- joint wheel3_barrel_4_joint: origin xyz=8.572527594031473e-19 -0.014 0.006 rpy=1.5707963267948966 0 -1.5707963267948966 -> xyz=2.2559282981050347e-18 -0.036842105 0.015789474 rpy=1.5707963267948966 0 -1.5707963267948966
- joint wheel3_barrel_5_joint: origin xyz=0.014 0.0 0.006 rpy=1.5707963267948966 0 0 -> xyz=0.036842105 0.0 0.015789474 rpy=1.5707963267948966 0 0
- joint wheel3_barrel_6_joint: origin xyz=8.572527594031473e-19 0.014 0.006 rpy=1.5707963267948966 0 1.5707963267948966 -> xyz=2.2559282981050347e-18 0.036842105 0.015789474 rpy=1.5707963267948966 0 1.5707963267948966
- joint wheel3_barrel_7_joint: origin xyz=-0.014 1.7145055188062945e-18 0.006 rpy=1.5707963267948966 0 3.141592653589793 -> xyz=-0.036842105 4.5118565962100695e-18 0.015789474 rpy=1.5707963267948966 0 3.141592653589793
- joint wheel3_barrel_8_joint: origin xyz=8.572527594031473e-19 -0.014 0.006 rpy=1.5707963267948966 0 -1.5707963267948966 -> xyz=2.2559282981050347e-18 -0.036842105 0.015789474 rpy=1.5707963267948966 0 -1.5707963267948966

File: models/omni_robot/omni_wheel.xacro (robot description, xacro)
@@ -5,5 +5,6 @@
       <parent link="${parent}"/>
       <child link="${prefix}_link"/>
-      <origin rpy="${pi/2} 0 ${dir}" xyz="${0.014*cos(dir)} ${0.014*sin(dir)} 0.006"/>
+      <!-- <origin rpy="${pi/2} 0 ${dir}" xyz="${0.014*cos(dir)} ${0.014*sin(dir)} 0.006"/> -->
+      <origin rpy="${pi/2} 0 ${dir}" xyz="${0.036842105*cos(dir)} ${0.036842105*sin(dir)} 0.015789474"/>
       <axis xyz="0 0 1"/>
       <dynamics damping="0.001"/>
@@ -22,5 +23,5 @@
       <visual>
         <geometry>
-          <mesh filename="model://omni_robot/meshes/omni_barrel.stl"/>
+          <mesh filename="model://omni_robot/meshes/omni_barrel100.stl"/>
         </geometry>
         <material name="black"/>
@@ -28,5 +29,5 @@
       <collision>
         <geometry>
-          <mesh filename="model://omni_robot/meshes/omni_barrel.stl"/>
+          <mesh filename="model://omni_robot/meshes/omni_barrel100.stl"/>
         </geometry>
       </collision>
@@ -136,5 +137,5 @@
       <visual>
         <geometry>
-          <mesh filename="model://omni_robot/meshes/omni_housing.stl"/>
+          <mesh filename="model://omni_robot/meshes/omni_housing100.stl"/>
         </geometry>
         <origin xyz="0 0 0" rpy="0 0 0"/>

File: models/omni_robot/urdf/omni_robot.xacro (robot description, xacro)
@@ -9,5 +9,6 @@
   <xacro:property name="wheel2_angle_deg" value="225"/>
   <xacro:property name="wheel3_angle_deg" value="315"/>
-  <xacro:property name="wheel_mount_radius" value="0.2"/>
+  <xacro:property name="wheel_mount_radius" value="0.3"/>
+  <xacro:property name="wheel_mount_hight" value="-0.04"/>
   <link name="base_link"/>
   <joint name="body_joint" type="fixed">
@@ -46,5 +47,5 @@
       xyz="${wheel_mount_radius*cos(radians(wheel0_angle_deg))}
           ${wheel_mount_radius*sin(radians(wheel0_angle_deg))}
-          0.019"
+          ${wheel_mount_hight}"
       rpy="0 0 ${radians(wheel0_angle_deg)}"/>
   </joint>
@@ -57,5 +58,5 @@
       xyz="${wheel_mount_radius*cos(radians(wheel1_angle_deg))}
           ${wheel_mount_radius*sin(radians(wheel1_angle_deg))}
-          0.019"
+          ${wheel_mount_hight}"
       rpy="0 0 ${radians(wheel1_angle_deg)}"/>
   </joint>
@@ -68,5 +69,5 @@
       xyz="${wheel_mount_radius*cos(radians(wheel2_angle_deg))}
           ${wheel_mount_radius*sin(radians(wheel2_angle_deg))}
-          0.019"
+          ${wheel_mount_hight}"
       rpy="0 0 ${radians(wheel2_angle_deg)}"/>
   </joint>
@@ -79,5 +80,5 @@
   xyz="${wheel_mount_radius*cos(radians(wheel3_angle_deg))}
        ${wheel_mount_radius*sin(radians(wheel3_angle_deg))}
-       0.019"
+       ${wheel_mount_hight}"
   rpy="0 0 ${radians(wheel3_angle_deg)}"/>
   </joint>

Commit message: Lidarの角度視野調整

File: models/omni_robot/omni_robot.urdf (robot description, URDF)
Before this commit: robot omni_robot, 91 links, 90 joints
Joints:
- joint lidar_joint: origin xyz=0 0 0.075 rpy=0 0 0 -> xyz=-0.3 0 -0.075 rpy=0 0 0
- joint wheel0_attach_joint: origin xyz=0.21213203435596426           0.21213203435596423           -0.04 rpy=0 0 0.7853981633974483 -> xyz=0.1767766952966369           0.17677669529663687           -0.04 rpy=0 0 0.7853981633974483
- joint wheel1_attach_joint: origin xyz=-0.21213203435596423           0.21213203435596426           -0.04 rpy=0 0 2.356194490192345 -> xyz=-0.17677669529663687           0.1767766952966369           -0.04 rpy=0 0 2.356194490192345
- joint wheel2_attach_joint: origin xyz=-0.2121320343559643           -0.21213203435596423           -0.04 rpy=0 0 3.9269908169872414 -> xyz=-0.17677669529663692           -0.17677669529663687           -0.04 rpy=0 0 3.9269908169872414
- joint wheel3_attach_joint: origin xyz=0.2121320343559642        -0.2121320343559643        -0.04 rpy=0 0 5.497787143782138 -> xyz=0.17677669529663684        -0.17677669529663692        -0.04 rpy=0 0 5.497787143782138

File: models/omni_robot/urdf/omni_robot.xacro (robot description, xacro)
@@ -9,5 +9,5 @@
   <xacro:property name="wheel2_angle_deg" value="225"/>
   <xacro:property name="wheel3_angle_deg" value="315"/>
-  <xacro:property name="wheel_mount_radius" value="0.3"/>
+  <xacro:property name="wheel_mount_radius" value="0.25"/>
   <xacro:property name="wheel_mount_hight" value="-0.04"/>
   <link name="base_link"/>
@@ -37,8 +37,8 @@
     prefix="lidar"
     parent="base_link"
-    xyz="0 0 0.075"
+    xyz="-0.3 0 -0.075"
     rpy="0 0 0"
-    angle_min="${-pi}"
-    angle_max="${pi}"/>
+    angle_min="${80 * pi / 180}"
+    angle_max="${280 * pi / 180}"/>
   <joint name="wheel0_attach_joint" type="fixed">
     <parent link="base_link"/>
