Commit message: でかいやつ正常に動いた

File: models/omni_robot/omni_common.xacro (robot description, xacro)
@@ -3,5 +3,5 @@
   <xacro:macro name="pi" params="3.1415926535897931" />
   <material name="gray">
-    <color rgba="0.8 0.8 0.8 1.0"/>
+    <color rgba="0.8 0.8 0.8 0.5"/>
   </material>
   <material name="black">
@@ -17,4 +17,7 @@
     <color rgba="1.0 0.5 0.5 1.0"/>
   </material>
+  <material name="green">
+    <color rgba="0 1.0 0 0.5"/>
+  </material>
   <material name="yellow">
     <color rgba="0 1.0 1.0 1.0"/>
