Commit message: omuni_nakamura_v11 wheelとbarrelがセットでstlになってるっぽい

File: models/omuni_nakamura_v11/urdf/materials.xacro (robot description, xacro)
@@ -1,6 +1,9 @@
 <?xml version="1.0" ?>
 <robot name="omuni_nakamura_v11" xmlns:xacro="http://www.ros.org/wiki/xacro" >
-<material name="silver_default">
-  <color rgba="0.700 0.700 0.700 1.000"/>
+<material name="orange">
+  <color rgba="1 0.42 0.12 0.85"/>
+</material>
+<material name="black">
+  <color rgba="0 0 0 1"/>
 </material>
 <material name="_">

File: models/omuni_nakamura_v11/urdf/omuni_nakamura_v11.xacro (robot description, xacro)
@@ -15,5 +15,5 @@
       <mesh filename="package://omuni_nakamura_v11/meshes/base_link.stl" scale="0.001 0.001 0.001"/>
     </geometry>
-    <material name="_"/>
+    <material name="orange"/>
   </visual>
   <collision>
@@ -115,5 +115,5 @@
       <mesh filename="package://omuni_nakamura_v11/meshes/omunimunimuni_v6_1.stl" scale="0.001 0.001 0.001"/>
     </geometry>
-    <material name="_"/>
+    <material name="black"/>
   </visual>
   <collision>
